Commit message: Lower G1-D arm mounts by 9.8 mm for torso frame alignment
G1-D torso_link is higher than G1 relative to the visual mesh; add
mount_xyz_* on UnitreeG1Arm and pass mount_xyz_z:=-0.0098 from G1-D.

Co-authored-by: Cursor <cursoragent@cursor.com>

File: unitree_g1_description/xacro/arm.xacro (robot description, xacro)
@@ -2,11 +2,10 @@
 <robot xmlns:xacro="http://www.ros.org/wiki/xacro">
 	<xacro:property name="PI" value="3.1415926535897931"/>
-	<xacro:macro name="UnitreeG1Arm" params="name direction:=1">
-		<!--
-		Unitree G1 Arm Macro
-		Parameters:
-		- name: arm name prefix (e.g., "left", "right")
-		- direction: 1 for right arm, -1 for left arm (for mirroring)
-		-->
+	<!--
+	mount_xyz_*: offset added to the nominal shoulder pitch origin on torso_link.
+	G1-D torso frame sits ~9.8 mm higher than G1's relative to the visual mesh;
+	pass mount_xyz_z:=-0.0098 so reused arms land on the G1-D torso.
+	-->
+	<xacro:macro name="UnitreeG1Arm" params="name direction:=1 parent:=torso_link mount_xyz_x:=0 mount_xyz_y:=0 mount_xyz_z:=0">
 		<xacro:property name="prefix" value="${name + '_' if name else ''}"/>
 		<!-- Shoulder Pitch Link -->
@@ -33,7 +32,7 @@
 		<!-- Shoulder Pitch Joint -->
 		<joint name="${prefix}shoulder_pitch_joint" type="revolute">
-			<origin xyz="0.0039563 ${direction*0.10022} 0.24778"
+			<origin xyz="${0.0039563 + mount_xyz_x} ${direction*0.10022 + mount_xyz_y} ${0.24778 + mount_xyz_z}"
 							rpy="${direction*0.27931} 5.4949E-05 ${direction*-0.00019159}"/>
-			<parent link="torso_link"/>
+			<parent link="${parent}"/>
 			<child link="${prefix}shoulder_pitch_link"/>
 			<axis xyz="0 1 0"/>

File: unitree_g1d_description/xacro/components/body.xacro (robot description, xacro)
@@ -4,20 +4,12 @@
 		<link name="logo_link">
 			<inertial>
-				<origin xyz="0 0 0" rpy="0 0 0"/>
 				<mass value="0.001"/>
 				<inertia ixx="1e-7" ixy="0" ixz="0" iyy="1e-7" iyz="0" izz="1e-7"/>
 			</inertial>
 			<visual>
-				<origin xyz="0 0 0" rpy="0 0 0"/>
 				<geometry>
 					<mesh filename="file://$(find unitree_g1d_description)/meshes/logo_link.STL"/>
 				</geometry>
 			</visual>
-			<collision>
-				<origin xyz="0 0 0" rpy="0 0 0"/>
-				<geometry>
-					<mesh filename="file://$(find unitree_g1d_description)/meshes/logo_link.STL"/>
-				</geometry>
-			</collision>
 		</link>
 		<link name="torso_link">
@@ -28,5 +20,4 @@
 			</inertial>
 			<visual>
-				<origin xyz="0 0 0" rpy="0 0 0"/>
 				<geometry>
 					<mesh filename="file://$(find unitree_g1d_description)/meshes/torso_link.STL"/>
@@ -34,5 +25,4 @@
 			</visual>
 			<collision>
-				<origin xyz="0 0 0" rpy="0 0 0"/>
 				<geometry>
 					<mesh filename="file://$(find unitree_g1d_description)/meshes/torso_link.STL"/>

File: unitree_g1d_description/xacro/components/chassis.xacro (robot description, xacro)
@@ -1,190 +1,182 @@
 <?xml version="1.0" ?>
 <robot xmlns:xacro="http://www.ros.org/wiki/xacro">
-	<xacro:macro name="UnitreeG1DChassis">
-		<link name="AGV_link">
-			<inertial>
-				<origin xyz="0 0 0" rpy="0 0 0"/>
-				<mass value="37"/>
-				<inertia ixx="0.091169133" ixy="0.000090756" ixz="0.000185579" iyy="0.081069202" iyz="-0.000057807" izz="0.158050329"/>
-			</inertial>
-			<visual>
-				<origin xyz="0 0 0" rpy="0 0 0"/>
-				<geometry>
-					<mesh filename="file://$(find unitree_g1d_description)/meshes/AGV_link.STL"/>
-				</geometry>
-			</visual>
-			<collision>
-				<origin xyz="0 0 0" rpy="0 0 0"/>
-				<geometry>
-					<mesh filename="file://$(find unitree_g1d_description)/meshes/AGV_link.STL"/>
-				</geometry>
-			</collision>
-		</link>
-		<link name="LZ_it_Link">
-			<inertial>
-				<origin xyz="-0.001566 -0.000192 -0.199159" rpy="0 0 0"/>
-				<mass value="3.4"/>
-				<inertia ixx="0.068209705" ixy="-0.00000153" ixz="0.000139907" iyy="0.068182916" iyz="-0.000006575" izz="0.010584232"/>
-			</inertial>
-			<visual>
-				<origin xyz="0 0 0" rpy="0 0 0"/>
-				<geometry>
-					<mesh filename="file://$(find unitree_g1d_description)/meshes/LZ_it_Link.STL"/>
-				</geometry>
-			</visual>
-		</link>
-		<link name="LZ_mt_Link">
-			<inertial>
-				<origin xyz="0.000494 -0.000062 0.216016" rpy="0 0 0"/>
-				<mass value="3.3"/>
-				<inertia ixx="0.057352663" ixy="0" ixz="0" iyy="0.05735287" iyz="0" izz="0.012847336"/>
-			</inertial>
-			<visual>
-				<origin xyz="0 0 0" rpy="0 0 0"/>
-				<geometry>
-					<mesh filename="file://$(find unitree_g1d_description)/meshes/LZ_mt_Link.STL"/>
-				</geometry>
-			</visual>
-		</link>
-		<link name="LZ_ot_Link">
-			<inertial>
-				<origin xyz="0.000375 0.000025 -0.000249652" rpy="0 0 0"/>
-				<mass value="3.3"/>
-				<inertia ixx="0.071819941" ixy="-0.000000949" ixz="-0.000008291" iyy="0.071821260" iyz="0.000015866" izz="0.014937474"/>
-			</inertial>
-			<visual>
-				<origin xyz="0 0 0" rpy="0 0 0"/>
-				<geometry>
-					<mesh filename="file://$(find unitree_g1d_description)/meshes/LZ_ot_Link.STL"/>
-				</geometry>
-			</visual>
-			<collision>
-				<origin xyz="0 0 0" rpy="0 0 0"/>
-				<geometry>
-					<mesh filename="file://$(find unitree_g1d_description)/meshes/LZ_ot_Link.STL"/>
-				</geometry>
-			</collision>
-		</link>
-		<link name="Left_Wheel_Link">
-			<inertial>
-				<origin xyz="-0.000003 -0.000309 -0.000002" rpy="0 0 0"/>
-				<mass value="1.5"/>
-				<inertia ixx="0.001541661" ixy="-0.000000034" ixz="0.00000004" iyy="0.002763727" iyz="-0.000000005" izz="0.001541722"/>
-			</inertial>
-			<visual>
-				<origin xyz="0 0 0" rpy="0 0 0"/>
-				<geometry>
-					<mesh filename="file://$(find unitree_g1d_description)/meshes/Left_Wheel_Link.STL"/>
-				</geometry>
-			</visual>
-			<collision>
-				<origin xyz="0 0 0" rpy="0 0 0"/>
-				<geometry>
-					<mesh filename="file://$(find unitree_g1d_description)/meshes/Left_Wheel_Link.STL"/>
-				</geometry>
-			</collision>
-		</link>
-		<link name="Pitching_Link">
-			<inertial>
-				<origin xyz="0.040544 -0.00377 0.051728" rpy="0 0 0"/>
-				<mass value="1.889"/>
-				<inertia ixx="0.003542953" ixy="0.000140065" ixz="-0.001148746" iyy="0.004845228" iyz="0.000090610" izz="0.003876594"/>
-			</inertial>
-			<visual>
-				<origin xyz="0 0 0" rpy="0 0 0"/>
-				<geometry>
-					<mesh filename="file://$(find unitree_g1d_description)/meshes/Pitching_Link.STL"/>
-				</geometry>
-			</visual>
-			<collision>
-				<origin xyz="0 0 0" rpy="0 0 0"/>
-				<geometry>
-					<mesh filename="file://$(find unitree_g1d_description)/meshes/Pitching_Link.STL"/>
-				</geometry>
-			</collision>
-		</link>
-		<link name="RIght_Wheel_Link">
-			<inertial>
-				<origin xyz="0.000003 0.000309 -0.000002" rpy="0 0 0"/>
-				<mass value="1.5"/>
-				<inertia ixx="0.001541661" ixy="-0.000000034" ixz="-0.000000004" iyy="0.002763727" iyz="0.000000005" izz="0.001541722"/>
-			</inertial>
-			<visual>
-				<origin xyz="0 0 0" rpy="0 0 0"/>
-				<geometry>
-					<mesh filename="file://$(find unitree_g1d_description)/meshes/RIght_Wheel_Link.STL"/>
-				</geometry>
-			</visual>
-			<collision>
-				<origin xyz="0 0 0" rpy="0 0 0"/>
-				<geometry>
-					<mesh filename="file://$(find unitree_g1d_description)/meshes/RIght_Wheel_Link.STL"/>
-				</geometry>
-			</collision>
-		</link>
-		<link name="Yaw_Link">
-			<inertial>
-				<origin xyz="0.000074 -0.000620 0.071221" rpy="0 0 0"/>
-				<mass value="1.144"/>
-				<inertia ixx="0.002602468" ixy="-0.000000583" ixz="-0.000000644" iyy="0.002202746" iyz="-0.000043725" izz="0.001228552"/>
-			</inertial>
-			<visual>
-				<origin xyz="0 0 0" rpy="0 0 0"/>
-				<geometry>
-					<mesh filename="file://$(find unitree_g1d_description)/meshes/Yaw_Link.STL"/>
-				</geometry>
-			</visual>
-			<collision>
-				<origin xyz="0 0 0" rpy="0 0 0"/>
-				<geometry>
-					<mesh filename="file://$(find unitree_g1d_description)/meshes/Yaw_Link.STL"/>
-				</geometry>
-			</collision>
-		</link>
-		<joint name="Left_Wheel_Joint" type="continuous">
-			<origin xyz="0.000225030065905006 0.2031 -0.0265" rpy="0 0 0"/>
-			<parent link="AGV_link"/>
-			<child link="Left_Wheel_Link"/>
-			<axis xyz="0 -1 0"/>
-			<limit lower="-3.1416" upper="3.1416" effort="8" velocity="100"/>
-		</joint>
-		<joint name="Right_Wheel_Joint" type="continuous">
-			<origin xyz="0.000225030065905024 -0.2031 -0.0265" rpy="0 0 0"/>
-			<parent link="AGV_link"/>
-			<child link="RIght_Wheel_Link"/>
-			<axis xyz="0 1 0"/>
-			<limit lower="-3.1416" upper="3.1416" effort="8" velocity="100"/>
-		</joint>
-		<joint name="LZ_ot_Joint" type="fixed">
-			<origin xyz="-0.000162639876214998 0 0.5275" rpy="0 0 0"/>
-			<parent link="AGV_link"/>
-			<child link="LZ_ot_Link"/>
-		</joint>
-		<joint name="LZ_mt_Joint" type="prismatic">
-			<origin xyz="0.000387669942120007 0 0.00999999999999995" rpy="0 0 0"/>
-			<parent link="LZ_ot_Link"/>
-			<child link="LZ_mt_Link"/>
-			<axis xyz="0 0 1"/>
-			<limit lower="0" upper="0.21" effort="500" velocity="0.05"/>
-		</joint>
-		<joint name="LZ_it_Joint" type="prismatic">
-			<origin xyz="0.0013627 0.00020167 0.018" rpy="0 0 0"/>
-			<parent link="LZ_mt_Link"/>
-			<child link="LZ_it_Link"/>
-			<axis xyz="0 0 1"/>
-			<limit lower="0" upper="0.21" effort="500" velocity="0.05"/>
-		</joint>
-		<joint name="Pitching_Joint" type="fixed">
-			<origin xyz="-0.0013627 -0.00020167 0.008" rpy="0 0 0"/>
-			<parent link="LZ_it_Link"/>
-			<child link="Pitching_Link"/>
-		</joint>
-		<joint name="Yaw_Joint" type="revolute">
-			<origin xyz="0.0555 0.0002165 0.066" rpy="0 0 0"/>
-			<parent link="Pitching_Link"/>
-			<child link="Yaw_Link"/>
-			<axis xyz="0 1 0"/>
-			<limit lower="-0.04363" upper="2.3562" effort="80" velocity="5"/>
-		</joint>
-	</xacro:macro>
+    <xacro:macro name="UnitreeG1DChassis">
+        <link name="AGV_link">
+            <inertial>
+                <mass value="37"/>
+                <inertia ixx="0.091169133" ixy="0.000090756" ixz="0.000185579" iyy="0.081069202" iyz="-0.000057807"
+                         izz="0.158050329"/>
+            </inertial>
+            <visual>
+                <geometry>
+                    <mesh filename="file://$(find unitree_g1d_description)/meshes/AGV_link.STL"/>
+                </geometry>
+            </visual>
+            <collision>
+                <geometry>
+                    <mesh filename="file://$(find unitree_g1d_description)/meshes/AGV_link.STL"/>
+                </geometry>
+            </collision>
+        </link>
+        <link name="LZ_it_Link">
+            <inertial>
+                <origin xyz="-0.001566 -0.000192 -0.199159"/>
+                <mass value="3.4"/>
+                <inertia ixx="0.068209705" ixy="-0.00000153" ixz="0.000139907" iyy="0.068182916" iyz="-0.000006575"
+                         izz="0.010584232"/>
+            </inertial>
+            <visual>
+                <geometry>
+                    <mesh filename="file://$(find unitree_g1d_description)/meshes/lz_it_link.glb"/>
+                </geometry>
+            </visual>
+        </link>
+        <link name="LZ_mt_Link">
+            <inertial>
+                <origin xyz="0.000494 -0.000062 0.216016"/>
+                <mass value="3.3"/>
+                <inertia ixx="0.057352663" ixy="0" ixz="0" iyy="0.05735287" iyz="0" izz="0.012847336"/>
+            </inertial>
+            <visual>
+                <geometry>
+                    <mesh filename="file://$(find unitree_g1d_description)/meshes/lz_mt_link.glb"/>
+                </geometry>
+            </visual>
+        </link>
+        <link name="LZ_ot_Link">
+            <inertial>
+                <origin xyz="0.000375 0.000025 -0.000249652"/>
+                <mass value="3.3"/>
+                <inertia ixx="0.071819941" ixy="-0.000000949" ixz="-0.000008291" iyy="0.071821260" iyz="0.000015866"
+                         izz="0.014937474"/>
+            </inertial>
+            <visual>
+                <geometry>
+                    <mesh filename="file://$(find unitree_g1d_description)/meshes/lz_ot_link.glb"/>
+                </geometry>
+            </visual>
+            <collision>
+                <geometry>
+                    <mesh filename="file://$(find unitree_g1d_description)/meshes/lz_ot_link.glb"/>
+                </geometry>
+            </collision>
+        </link>
+        <link name="Left_Wheel_Link">
+            <inertial>
+                <origin xyz="-0.000003 -0.000309 -0.000002"/>
+                <mass value="1.5"/>
+                <inertia ixx="0.001541661" ixy="-0.000000034" ixz="0.00000004" iyy="0.002763727" iyz="-0.000000005"
+                         izz="0.001541722"/>
+            </inertial>
+            <visual>
+                <geometry>
+                    <mesh filename="file://$(find unitree_g1d_description)/meshes/Left_Wheel_Link.STL"/>
+                </geometry>
+            </visual>
+            <collision>
+                <geometry>
+                    <mesh filename="file://$(find unitree_g1d_description)/meshes/Left_Wheel_Link.STL"/>
+                </geometry>
+            </collision>
+        </link>
+        <link name="Pitching_Link">
+            <inertial>
+                <origin xyz="0.040544 -0.00377 0.051728"/>
+                <mass value="1.889"/>
+                <inertia ixx="0.003542953" ixy="0.000140065" ixz="-0.001148746" iyy="0.004845228" iyz="0.000090610"
+                         izz="0.003876594"/>
+            </inertial>
+            <visual>
+                <geometry>
+                    <mesh filename="file://$(find unitree_g1d_description)/meshes/pitching_link.glb"/>
+                </geometry>
+            </visual>
+            <collision>
+                <geometry>
+                    <mesh filename="file://$(find unitree_g1d_description)/meshes/pitching_link.glb"/>
+                </geometry>
+            </collision>
+        </link>
+        <link name="RIght_Wheel_Link">
+            <inertial>
+                <origin xyz="0.000003 0.000309 -0.000002"/>
+                <mass value="1.5"/>
+                <inertia ixx="0.001541661" ixy="-0.000000034" ixz="-0.000000004" iyy="0.002763727" iyz="0.000000005"
+                         izz="0.001541722"/>
+            </inertial>
+            <visual>
+                <geometry>
+                    <mesh filename="file://$(find unitree_g1d_description)/meshes/RIght_Wheel_Link.STL"/>
+                </geometry>
+            </visual>
+            <collision>
+                <geometry>
+                    <mesh filename="file://$(find unitree_g1d_description)/meshes/RIght_Wheel_Link.STL"/>
+                </geometry>
+            </collision>
+        </link>
+        <link name="Yaw_Link">
+            <inertial>
+                <origin xyz="0.000074 -0.000620 0.071221"/>
+                <mass value="1.144"/>
+                <inertia ixx="0.002602468" ixy="-0.000000583" ixz="-0.000000644" iyy="0.002202746" iyz="-0.000043725"
+                         izz="0.001228552"/>
+            </inertial>
+            <visual>
+                <geometry>
+                    <mesh filename="file://$(find unitree_g1d_description)/meshes/yaw_link.glb"/>
+                </geometry>
+            </visual>
+            <collision>
+                <geometry>
+                    <mesh filename="file://$(find unitree_g1d_description)/meshes/yaw_link.glb"/>
+                </geometry>
+            </collision>
+        </link>
+        <joint name="Left_Wheel_Joint" type="continuous">
+            <origin xyz="0.000225030065905006 0.2031 -0.0265"/>
+            <parent link="AGV_link"/>
+            <child link="Left_Wheel_Link"/>
+            <axis xyz="0 -1 0"/>
+            <limit lower="-3.1416" upper="3.1416" effort="8" velocity="100"/>
+        </joint>
+        <joint name="Right_Wheel_Joint" type="continuous">
+            <origin xyz="0.000225030065905024 -0.2031 -0.0265"/>
+            <parent link="AGV_link"/>
+            <child link="RIght_Wheel_Link"/>
+            <axis xyz="0 1 0"/>
+            <limit lower="-3.1416" upper="3.1416" effort="8" velocity="100"/>
+        </joint>
+        <joint name="LZ_ot_Joint" type="fixed">
+            <origin xyz="-0.000162639876214998 0 0.5275"/>
+            <parent link="AGV_link"/>
+            <child link="LZ_ot_Link"/>
+        </joint>
+        <joint name="LZ_mt_Joint" type="prismatic">
+            <origin xyz="0.000387669942120007 0 0.00999999999999995"/>
+            <parent link="LZ_ot_Link"/>
+            <child link="LZ_mt_Link"/>
+            <axis xyz="0 0 1"/>
+            <limit lower="0" upper="0.21" effort="500" velocity="0.05"/>
+        </joint>
+        <joint name="LZ_it_Joint" type="prismatic">
+            <origin xyz="0.0013627 0.00020167 0.018"/>
+            <parent link="LZ_mt_Link"/>
+            <child link="LZ_it_Link"/>
+            <axis xyz="0 0 1"/>
+            <limit lower="0" upper="0.21" effort="500" velocity="0.05"/>
+        </joint>
+        <joint name="Pitching_Joint" type="fixed">
+            <origin xyz="-0.0013627 -0.00020167 0.008"/>
+            <parent link="LZ_it_Link"/>
+            <child link="Pitching_Link"/>
+        </joint>
+        <joint name="Yaw_Joint" type="revolute">
+            <origin xyz="0.0555 0.0002165 0.066"/>
+            <parent link="Pitching_Link"/>
+            <child link="Yaw_Link"/>
+            <axis xyz="0 1 0"/>
+            <limit lower="-0.04363" upper="2.3562" effort="80" velocity="5"/>
+        </joint>
+    </xacro:macro>
 </robot>

File: unitree_g1d_description/xacro/robot.xacro (robot description, xacro)
@@ -6,11 +6,11 @@
 	<xacro:UnitreeG1DChassis/>
 	<xacro:UnitreeG1DBody/>
-	<!-- Shared G1 head (G1-D mount is 10 mm lower) -->
+	<!-- Shared G1 head (official G1-D mount is 10 mm lower than G1) -->
 	<xacro:include filename="$(find unitree_g1_description)/xacro/head.xacro"/>
 	<xacro:UnitreeG1Head xyz_z="-0.054"/>
-	<!-- Shared G1 arms -->
+	<!-- Shared G1 arms: G1-D torso_link is 9.8 mm higher vs G1 mesh alignment -->
 	<xacro:include filename="$(find unitree_g1_description)/xacro/arm.xacro"/>
-	<xacro:UnitreeG1Arm name="left" direction="1"/>
-	<xacro:UnitreeG1Arm name="right" direction="-1"/>
+	<xacro:UnitreeG1Arm name="left" direction="1" mount_xyz_z="-0.0098"/>
+	<xacro:UnitreeG1Arm name="right" direction="-1" mount_xyz_z="-0.0098"/>
 	<!-- Shared G1 end effectors (default Dex3) -->
 	<xacro:include filename="$(find unitree_g1_description)/xacro/hand.xacro"/>
