Commit message: add glb mesh

File: unitree_g1_description/xacro/arm.xacro (robot description, xacro)
@@ -19,5 +19,5 @@
 			<visual>
 				<geometry>
-					<mesh filename="file://$(find unitree_g1_description)/meshes/arm/shoulder_pitch.obj"
+					<mesh filename="file://$(find unitree_g1_description)/meshes/arm/shoulder_pitch.glb"
 								scale="1 ${direction} 1"/>
 				</geometry>
@@ -49,5 +49,5 @@
 			<visual>
 				<geometry>
-					<mesh filename="file://$(find unitree_g1_description)/meshes/arm/shoulder_roll.obj"
+					<mesh filename="file://$(find unitree_g1_description)/meshes/arm/shoulder_roll.glb"
 								scale="1 ${direction} 1"/>
 				</geometry>
@@ -79,5 +79,5 @@
 			<visual>
 				<geometry>
-					<mesh filename="file://$(find unitree_g1_description)/meshes/arm/shoulder_yaw.obj"
+					<mesh filename="file://$(find unitree_g1_description)/meshes/arm/shoulder_yaw.glb"
 								scale="1 ${direction} 1"/>
 				</geometry>
@@ -114,5 +114,5 @@
 			<visual>
 				<geometry>
-					<mesh filename="file://$(find unitree_g1_description)/meshes/arm/elbow.obj"
+					<mesh filename="file://$(find unitree_g1_description)/meshes/arm/elbow.glb"
 								scale="1 ${direction} 1"/>
 				</geometry>
@@ -144,5 +144,6 @@
 			<visual>
 				<geometry>
-					<mesh filename="file://$(find unitree_g1_description)/meshes/arm/wrist_roll.obj"/>
+					<mesh filename="file://$(find unitree_g1_description)/meshes/arm/wrist_roll.glb"
+								scale="1 ${direction} 1"/>
 				</geometry>
 			</visual>
@@ -167,5 +168,6 @@
 			<visual>
 				<geometry>
-					<mesh filename="file://$(find unitree_g1_description)/meshes/arm/wrist_pitch.obj"/>
+					<mesh filename="file://$(find unitree_g1_description)/meshes/arm/wrist_pitch.glb"
+								scale="1 ${direction} 1"/>
 				</geometry>
 			</visual>
@@ -202,5 +204,5 @@
 			<visual>
 				<geometry>
-					<mesh filename="file://$(find unitree_g1_description)/meshes/arm/wrist_yaw.obj" scale="1 ${direction} 1"/>
+					<mesh filename="file://$(find unitree_g1_description)/meshes/arm/wrist_yaw.glb" scale="1 ${direction} 1"/>
 				</geometry>
 			</visual>

File: unitree_g1_description/xacro/body.xacro (robot description, xacro)
@@ -1,74 +1,75 @@
 <?xml version="1.0" ?>
 <robot xmlns:xacro="http://www.ros.org/wiki/xacro">
-	<xacro:include filename="$(find unitree_g1_description)/xacro/torso.xacro"/>
-	<xacro:macro name="UnitreeG1Body">
-		<!-- Pelvis + 3-DoF waist; torso/logo/sensors via UnitreeG1Torso -->
-		<link name="base_link"/>
-		<joint name="base_link_joint" type="fixed">
-			<parent link="base_link"/>
-			<child link="pelvis"/>
-		</joint>
-		<link name="pelvis">
-			<inertial>
-				<origin xyz="0 0 -0.07605"/>
-				<mass value="3.813"/>
-				<inertia ixx="0.010549" ixy="0" ixz="2.1E-06" iyy="0.0093089" iyz="0" izz="0.0079184"/>
-			</inertial>
-			<visual>
-				<geometry>
-					<mesh filename="file://$(find unitree_g1_description)/meshes/body/pelvis.obj"/>
-				</geometry>
-			</visual>
-		</link>
-		<link name="waist_yaw_link">
-			<inertial>
-				<origin xyz="0.003494 0.000233 0.018034"/>
-				<mass value="0.214"/>
-				<inertia ixx="0.00010673" ixy="2.703E-06" ixz="-7.631E-06" iyy="0.00010422" iyz="-2.01E-07" izz="0.0001625"/>
-			</inertial>
-			<visual>
-				<geometry>
-					<mesh filename="file://$(find unitree_g1_description)/meshes/body/waist_yaw.obj"/>
-				</geometry>
-			</visual>
-		</link>
-		<joint name="waist_yaw_joint" type="revolute">
-			<parent link="pelvis"/>
-			<child link="waist_yaw_link"/>
-			<axis xyz="0 0 1"/>
-			<limit lower="-2.618" upper="2.618" effort="88" velocity="32"/>
-		</joint>
-		<link name="waist_roll_link">
-			<inertial>
-				<origin xyz="0 2.3E-05 0"/>
-				<mass value="0.086"/>
-				<inertia ixx="7.079E-06" ixy="0" ixz="0" iyy="6.339E-06" iyz="0" izz="8.245E-06"/>
-			</inertial>
-			<visual>
-				<geometry>
-					<mesh filename="file://$(find unitree_g1_description)/meshes/body/waist_roll.obj"/>
-				</geometry>
-			</visual>
-		</link>
-		<joint name="waist_roll_joint" type="revolute">
-			<origin xyz="-0.0039635 0 0.044"/>
-			<parent link="waist_yaw_link"/>
-			<child link="waist_roll_link"/>
-			<axis xyz="1 0 0"/>
-			<limit lower="-0.52" upper="0.52" effort="35" velocity="30"/>
-		</joint>
-		<xacro:UnitreeG1Torso/>
-		<joint name="waist_pitch_joint" type="revolute">
-			<parent link="waist_roll_link"/>
-			<child link="torso_link"/>
-			<axis xyz="0 1 0"/>
-			<limit lower="-0.52" upper="0.52" effort="35" velocity="30"/>
-		</joint>
-		<link name="imu_in_pelvis"/>
-		<joint name="imu_in_pelvis_joint" type="fixed">
-			<origin xyz="0.04525 0 -0.08339"/>
-			<parent link="pelvis"/>
-			<child link="imu_in_pelvis"/>
-		</joint>
-	</xacro:macro>
+    <xacro:include filename="$(find unitree_g1_description)/xacro/torso.xacro"/>
+    <xacro:macro name="UnitreeG1Body">
+        <!-- Pelvis + 3-DoF waist; torso/logo/sensors via UnitreeG1Torso -->
+        <link name="base_link"/>
+        <joint name="base_link_joint" type="fixed">
+            <parent link="base_link"/>
+            <child link="pelvis"/>
+        </joint>
+        <link name="pelvis">
+            <inertial>
+                <origin xyz="0 0 -0.07605"/>
+                <mass value="3.813"/>
+                <inertia ixx="0.010549" ixy="0" ixz="2.1E-06" iyy="0.0093089" iyz="0" izz="0.0079184"/>
+            </inertial>
+            <visual>
+                <geometry>
+                    <mesh filename="file://$(find unitree_g1_description)/meshes/body/pelvis.glb"/>
+                </geometry>
+            </visual>
+        </link>
+        <link name="waist_yaw_link">
+            <inertial>
+                <origin xyz="0.003494 0.000233 0.018034"/>
+                <mass value="0.214"/>
+                <inertia ixx="0.00010673" ixy="2.703E-06" ixz="-7.631E-06" iyy="0.00010422" iyz="-2.01E-07"
+                         izz="0.0001625"/>
+            </inertial>
+            <visual>
+                <geometry>
+                    <mesh filename="file://$(find unitree_g1_description)/meshes/body/waist_yaw.glb"/>
+                </geometry>
+            </visual>
+        </link>
+        <joint name="waist_yaw_joint" type="revolute">
+            <parent link="pelvis"/>
+            <child link="waist_yaw_link"/>
+            <axis xyz="0 0 1"/>
+            <limit lower="-2.618" upper="2.618" effort="88" velocity="32"/>
+        </joint>
+        <link name="waist_roll_link">
+            <inertial>
+                <origin xyz="0 2.3E-05 0"/>
+                <mass value="0.086"/>
+                <inertia ixx="7.079E-06" ixy="0" ixz="0" iyy="6.339E-06" iyz="0" izz="8.245E-06"/>
+            </inertial>
+            <visual>
+                <geometry>
+                    <mesh filename="file://$(find unitree_g1_description)/meshes/body/waist_roll.glb"/>
+                </geometry>
+            </visual>
+        </link>
+        <joint name="waist_roll_joint" type="revolute">
+            <origin xyz="-0.0039635 0 0.044"/>
+            <parent link="waist_yaw_link"/>
+            <child link="waist_roll_link"/>
+            <axis xyz="1 0 0"/>
+            <limit lower="-0.52" upper="0.52" effort="35" velocity="30"/>
+        </joint>
+        <xacro:UnitreeG1Torso/>
+        <joint name="waist_pitch_joint" type="revolute">
+            <parent link="waist_roll_link"/>
+            <child link="torso_link"/>
+            <axis xyz="0 1 0"/>
+            <limit lower="-0.52" upper="0.52" effort="35" velocity="30"/>
+        </joint>
+        <link name="imu_in_pelvis"/>
+        <joint name="imu_in_pelvis_joint" type="fixed">
+            <origin xyz="0.04525 0 -0.08339"/>
+            <parent link="pelvis"/>
+            <child link="imu_in_pelvis"/>
+        </joint>
+    </xacro:macro>
 </robot>

File: unitree_g1_description/xacro/eefs.xacro (robot description, xacro)
@@ -28,5 +28,5 @@
 					<visual>
 						<geometry>
-							<mesh filename="file://$(find unitree_g1_description)/meshes/arm/hand.obj" scale="1 ${direction} 1"/>
+							<mesh filename="file://$(find unitree_g1_description)/meshes/arm/hand.glb" scale="1 ${direction} 1"/>
 						</geometry>
 					</visual>

File: unitree_g1_description/xacro/head.xacro (robot description, xacro)
@@ -15,10 +15,10 @@
 			<visual>
 				<geometry>
-					<mesh filename="file://$(find unitree_g1_description)/meshes/body/head.obj"/>
+					<mesh filename="file://$(find unitree_g1_description)/meshes/body/head.glb"/>
 				</geometry>
 			</visual>
 			<collision>
 				<geometry>
-					<mesh filename="file://$(find unitree_g1_description)/meshes/body/head.obj"/>
+					<mesh filename="file://$(find unitree_g1_description)/meshes/body/head.glb"/>
 				</geometry>
 			</collision>

File: unitree_g1_description/xacro/leg.xacro (robot description, xacro)
@@ -13,5 +13,5 @@
 			<visual>
 				<geometry>
-					<mesh filename="file://$(find unitree_g1_description)/meshes/leg/hip_pitch.obj"
+					<mesh filename="file://$(find unitree_g1_description)/meshes/leg/hip_pitch.glb"
 								scale="1 ${direction} 1"/>
 				</geometry>
@@ -19,5 +19,5 @@
 			<collision>
 				<geometry>
-					<mesh filename="file://$(find unitree_g1_description)/meshes/leg/hip_pitch.obj"
+					<mesh filename="file://$(find unitree_g1_description)/meshes/leg/hip_pitch.glb"
 								scale="1 ${direction} 1"/>
 				</geometry>
@@ -42,10 +42,12 @@
 			<visual>
 				<geometry>
-					<mesh filename="file://$(find unitree_g1_description)/meshes/leg/hip_roll.obj"/>
+					<mesh filename="file://$(find unitree_g1_description)/meshes/leg/hip_roll.glb"
+								scale="1 ${direction} 1"/>
 				</geometry>
 			</visual>
 			<collision>
 				<geometry>
-					<mesh filename="file://$(find unitree_g1_description)/meshes/leg/hip_roll.obj"/>
+					<mesh filename="file://$(find unitree_g1_description)/meshes/leg/hip_roll.glb"
+								scale="1 ${direction} 1"/>
 				</geometry>
 			</collision>
@@ -70,5 +72,5 @@
 			<visual>
 				<geometry>
-					<mesh filename="file://$(find unitree_g1_description)/meshes/leg/hip_yaw.obj"
+					<mesh filename="file://$(find unitree_g1_description)/meshes/leg/hip_yaw.glb"
 								scale="1 ${direction} 1"/>
 				</geometry>
@@ -76,5 +78,5 @@
 			<collision>
 				<geometry>
-					<mesh filename="file://$(find unitree_g1_description)/meshes/leg/hip_yaw.obj"
+					<mesh filename="file://$(find unitree_g1_description)/meshes/leg/hip_yaw.glb"
 								scale="1 ${direction} 1"/>
 				</geometry>
@@ -99,5 +101,5 @@
 			<visual>
 				<geometry>
-					<mesh filename="file://$(find unitree_g1_description)/meshes/leg/knee.obj"
+					<mesh filename="file://$(find unitree_g1_description)/meshes/leg/knee.glb"
 								scale="1 ${direction} 1"/>
 				</geometry>
@@ -105,5 +107,5 @@
 			<collision>
 				<geometry>
-					<mesh filename="file://$(find unitree_g1_description)/meshes/leg/knee.obj"
+					<mesh filename="file://$(find unitree_g1_description)/meshes/leg/knee.glb"
 								scale="1 ${direction} 1"/>
 				</geometry>
@@ -127,10 +129,12 @@
 			<visual>
 				<geometry>
-					<mesh filename="file://$(find unitree_g1_description)/meshes/leg/ankle_pitch.obj"/>
+					<mesh filename="file://$(find unitree_g1_description)/meshes/leg/ankle_pitch.glb"
+								scale="1 ${direction} 1"/>
 				</geometry>
 			</visual>
 			<collision>
 				<geometry>
-					<mesh filename="file://$(find unitree_g1_description)/meshes/leg/ankle_pitch.obj"/>
+					<mesh filename="file://$(find unitree_g1_description)/meshes/leg/ankle_pitch.glb"
+								scale="1 ${direction} 1"/>
 				</geometry>
 			</collision>
@@ -154,5 +158,6 @@
 			<visual>
 				<geometry>
-					<mesh filename="file://$(find unitree_g1_description)/meshes/leg/ankle_roll.obj"/>
+					<mesh filename="file://$(find unitree_g1_description)/meshes/leg/ankle_roll.glb"
+								scale="1 ${direction} 1"/>
 				</geometry>
 			</visual>

File: unitree_g1_description/xacro/torso.xacro (robot description, xacro)
@@ -16,5 +16,5 @@
 			<visual>
 				<geometry>
-					<mesh filename="file://$(find unitree_g1_description)/meshes/body/torso.obj"/>
+					<mesh filename="file://$(find unitree_g1_description)/meshes/body/torso.glb"/>
 				</geometry>
 			</visual>
@@ -39,5 +39,5 @@
 			<visual>
 				<geometry>
-					<mesh filename="file://$(find unitree_g1_description)/meshes/body/logo.obj"/>
+					<mesh filename="file://$(find unitree_g1_description)/meshes/body/logo.glb"/>
 				</geometry>
 			</visual>

File: unitree_g1d_description/xacro/component.xacro (robot description, xacro)
@@ -20,5 +20,5 @@
 	</xacro:if>
 	<xacro:if value="${'$(arg type)' == 'body'}">
-		<link name="Yaw_Link"/>
+		<link name="waist_pitch_link"/>
 		<xacro:UnitreeG1DBody/>
 	</xacro:if>

File: unitree_g1d_description/xacro/components/body.xacro (robot description, xacro)
@@ -9,7 +9,7 @@
 	<xacro:macro name="UnitreeG1DBody">
 		<xacro:UnitreeG1Torso/>
-		<joint name="torso_yaw_joint" type="revolute">
+		<joint name="waist_yaw_joint" type="revolute">
 			<origin xyz="-0.0023536 -0.000048782 ${0.104008566 - 0.0098}" rpy="0 0 0"/>
-			<parent link="Yaw_Link"/>
+			<parent link="waist_pitch_link"/>
 			<child link="torso_link"/>
 			<axis xyz="0 0 1"/>

File: unitree_g1d_description/xacro/components/chassis.xacro (robot description, xacro)
@@ -166,5 +166,5 @@
 			<parent link="AGV_link"/>
 			<child link="Left_Wheel_Link"/>
-			<axis xyz="0 -1 0"/>
+			<axis xyz="0 1 0"/>
 			<limit lower="-3.1416" upper="3.1416" effort="8" velocity="100"/>
 		</joint>

File: unitree_g1d_description/xacro/components/lift.xacro (robot description, xacro)
@@ -1,6 +1,6 @@
 <?xml version="1.0" ?>
 <robot xmlns:xacro="http://www.ros.org/wiki/xacro">
-	<!-- 3-stage lift column (LZ_*) + waist pitch/yaw stage (Pitching / Yaw).
-	     Attaches to AGV_link; body mounts on Yaw_Link. -->
+	<!-- 3-stage lift column (LZ_*) + waist pitch/yaw stage (waist_mount fixed + waist_pitch_joint; official CAD names Pitching_/Yaw_*).
+	     Attaches to AGV_link; body mounts on waist_pitch_link. -->
 	<xacro:macro name="UnitreeG1DLift">
 		<link name="LZ_ot_Link">
@@ -33,4 +33,9 @@
 				</geometry>
 			</visual>
+			<collision>
+				<geometry>
+					<mesh filename="file://$(find unitree_g1d_description)/meshes/lz_mt_link.glb"/>
+				</geometry>
+			</collision>
 		</link>
 		<link name="LZ_it_Link">
@@ -46,6 +51,11 @@
 				</geometry>
 			</visual>
+			<collision>
+				<geometry>
+					<mesh filename="file://$(find unitree_g1d_description)/meshes/lz_it_link.glb"/>
+				</geometry>
+			</collision>
 		</link>
-		<link name="Pitching_Link">
+		<link name="waist_mount_link">
 			<inertial>
 				<origin xyz="0.040544 -0.00377 0.051728"/>
@@ -65,5 +75,5 @@
 			</collision>
 		</link>
-		<link name="Yaw_Link">
+		<link name="waist_pitch_link">
 			<inertial>
 				<origin xyz="0.000074 -0.000620 0.071221"/>
@@ -102,13 +112,13 @@
 			<limit lower="0" upper="0.21" effort="500" velocity="0.05"/>
 		</joint>
-		<joint name="Pitching_Joint" type="fixed">
+		<joint name="waist_mount_joint" type="fixed">
 			<origin xyz="-0.0013627 -0.00020167 0.008"/>
 			<parent link="LZ_it_Link"/>
-			<child link="Pitching_Link"/>
+			<child link="waist_mount_link"/>
 		</joint>
-		<joint name="Yaw_Joint" type="revolute">
+		<joint name="waist_pitch_joint" type="revolute">
 			<origin xyz="0.0555 0.0002165 0.066"/>
-			<parent link="Pitching_Link"/>
-			<child link="Yaw_Link"/>
+			<parent link="waist_mount_link"/>
+			<child link="waist_pitch_link"/>
 			<axis xyz="0 1 0"/>
 			<limit lower="-0.04363" upper="2.3562" effort="80" velocity="5"/>

File: unitree_g1d_description/xacro/ros2_control/robot.xacro (robot description, xacro)
@@ -55,5 +55,5 @@
 			<state_interface name="effort"/>
 		</joint>
-		<joint name="Yaw_Joint">
+		<joint name="waist_pitch_joint">
 			<command_interface name="position"/>
 			<state_interface name="position"/>
@@ -61,5 +61,5 @@
 			<state_interface name="effort"/>
 		</joint>
-		<joint name="torso_yaw_joint">
+		<joint name="waist_yaw_joint">
 			<command_interface name="position"/>
 			<state_interface name="position"/>
