Commit message: Reuse G1 torso and logo on G1-D with adjusted yaw mount
Extract UnitreeG1Torso, mount it from Yaw_Link via torso_yaw_joint with
z reduced by 9.8 mm, and drop G1-D-specific arm/head offsets and meshes.

Co-authored-by: Cursor <cursoragent@cursor.com>

File: unitree_g1_description/xacro/body.xacro (robot description, xacro)
@@ -1,9 +1,7 @@
 <?xml version="1.0" ?>
 <robot xmlns:xacro="http://www.ros.org/wiki/xacro">
+	<xacro:include filename="$(find unitree_g1_description)/xacro/torso.xacro"/>
 	<xacro:macro name="UnitreeG1Body">
-		<!--
-		Unitree G1 Body Macro
-		Includes: pelvis, torso, head, sensors, and logo
-		-->
+		<!-- Pelvis + 3-DoF waist; torso/logo/sensors via UnitreeG1Torso -->
 		<link name="base_link"/>
 		<joint name="base_link_joint" type="fixed">
@@ -11,5 +9,4 @@
 			<child link="pelvis"/>
 		</joint>
-		<!-- Pelvis Link -->
 		<link name="pelvis">
 			<inertial>
@@ -24,6 +21,4 @@
 			</visual>
 		</link>
-		<!-- Torso Structure -->
-		<!-- Waist Yaw Link -->
 		<link name="waist_yaw_link">
 			<inertial>
@@ -38,5 +33,4 @@
 			</visual>
 		</link>
-		<!-- Waist Yaw Joint -->
 		<joint name="waist_yaw_joint" type="revolute">
 			<parent link="pelvis"/>
@@ -45,5 +39,4 @@
 			<limit lower="-2.618" upper="2.618" effort="88" velocity="32"/>
 		</joint>
-		<!-- Waist Roll Link -->
 		<link name="waist_roll_link">
 			<inertial>
@@ -58,5 +51,4 @@
 			</visual>
 		</link>
-		<!-- Waist Roll Joint -->
 		<joint name="waist_roll_joint" type="revolute">
 			<origin xyz="-0.0039635 0 0.044"/>
@@ -66,30 +58,5 @@
 			<limit lower="-0.52" upper="0.52" effort="35" velocity="30"/>
 		</joint>
-		<!-- Torso Link -->
-		<link name="torso_link">
-			<inertial>
-				<origin xyz="0.000931 0.000346 0.15082"/>
-				<mass value="6.78"/>
-				<inertia ixx="0.05905" ixy="3.3302E-05" ixz="-0.0017715" iyy="0.047014" iyz="-2.2399E-05" izz="0.025652"/>
-			</inertial>
-			<visual>
-				<geometry>
-					<mesh filename="file://$(find unitree_g1_description)/meshes/body/torso.obj"/>
-				</geometry>
-			</visual>
-			<collision>
-				<origin xyz="0.008 0 0.05"/>
-				<geometry>
-					<box size="0.12 0.15 0.15"/>
-				</geometry>
-			</collision>
-			<collision>
-				<origin xyz="0.008 0 0.2"/>
-				<geometry>
-					<box size="0.12 0.2 0.15"/>
-				</geometry>
-			</collision>
-		</link>
-		<!-- Waist Pitch Joint -->
+		<xacro:UnitreeG1Torso/>
 		<joint name="waist_pitch_joint" type="revolute">
 			<parent link="waist_roll_link"/>
@@ -97,29 +64,4 @@
 			<axis xyz="0 1 0"/>
 			<limit lower="-0.52" upper="0.52" effort="35" velocity="30"/>
-		</joint>
-		<!-- Logo -->
-		<link name="logo_link">
-			<inertial>
-				<mass value="0.001"/>
-				<inertia ixx="1e-7" ixy="0" ixz="0" iyy="1e-7" iyz="0" izz="1e-7"/>
-			</inertial>
-			<visual>
-				<geometry>
-					<mesh filename="file://$(find unitree_g1_description)/meshes/body/logo.obj"/>
-				</geometry>
-			</visual>
-		</link>
-		<joint name="logo_joint" type="fixed">
-			<origin xyz="0.0039635 0 -0.044"/>
-			<parent link="torso_link"/>
-			<child link="logo_link"/>
-		</joint>
-		<!-- Head is in head.xacro (UnitreeG1Head); instantiated from robot.xacro -->
-		<!-- IMU Sensors -->
-		<link name="imu_in_torso"/>
-		<joint name="imu_in_torso_joint" type="fixed">
-			<origin xyz="-0.03959 -0.00224 0.14792"/>
-			<parent link="torso_link"/>
-			<child link="imu_in_torso"/>
 		</joint>
 		<link name="imu_in_pelvis"/>
@@ -129,17 +71,4 @@
 			<child link="imu_in_pelvis"/>
 		</joint>
-		<!-- Cameras and Sensors -->
-		<link name="d435_link"/>
-		<joint name="d435_joint" type="fixed">
-			<origin xyz="0.0576235 0.01753 0.42987" rpy="0 0.8307767239493009 0"/>
-			<parent link="torso_link"/>
-			<child link="d435_link"/>
-		</joint>
-		<link name="mid360_link"/>
-		<joint name="mid360_joint" type="fixed">
-			<origin xyz="0.0002835 0.00003 0.41618" rpy="0 0.04014257279586953 0"/>
-			<parent link="torso_link"/>
-			<child link="mid360_link"/>
-		</joint>
 	</xacro:macro>
 </robot>

File: unitree_g1d_description/xacro/components/body.xacro (robot description, xacro)
@@ -1,35 +1,14 @@
 <?xml version="1.0" ?>
 <robot xmlns:xacro="http://www.ros.org/wiki/xacro">
+	<xacro:include filename="$(find unitree_g1_description)/xacro/torso.xacro"/>
+	<!--
+	Mount G1 torso onto the G1-D yaw stage.
+	Official torso_Joint origin was z=0.104008566 for the G1-D torso frame;
+	G1 torso_link is 9.8 mm lower relative to the visual mesh, so subtract that.
+	-->
 	<xacro:macro name="UnitreeG1DBody">
-		<link name="logo_link">
-			<inertial>
-				<mass value="0.001"/>
-				<inertia ixx="1e-7" ixy="0" ixz="0" iyy="1e-7" iyz="0" izz="1e-7"/>
-			</inertial>
-			<visual>
-				<geometry>
-					<mesh filename="file://$(find unitree_g1d_description)/meshes/logo_link.STL"/>
-				</geometry>
-			</visual>
-		</link>
-		<link name="torso_link">
-			<inertial>
-				<origin xyz="0.002601 0.000257 0.153719" rpy="0 0 0"/>
-				<mass value="8.562"/>
-				<inertia ixx="0.065674966" ixy="-8.597E-05" ixz="-0.001737252" iyy="0.053535188" iyz="8.6899E-05" izz="0.030808125"/>
-			</inertial>
-			<visual>
-				<geometry>
-					<mesh filename="file://$(find unitree_g1d_description)/meshes/torso_link.STL"/>
-				</geometry>
-			</visual>
-			<collision>
-				<geometry>
-					<mesh filename="file://$(find unitree_g1d_description)/meshes/torso_link.STL"/>
-				</geometry>
-			</collision>
-		</link>
-		<joint name="torso_Joint" type="revolute">
-			<origin xyz="-0.0023536 -0.000048782 0.104008566" rpy="0 0 0"/>
+		<xacro:UnitreeG1Torso/>
+		<joint name="torso_yaw_joint" type="revolute">
+			<origin xyz="-0.0023536 -0.000048782 ${0.104008566 - 0.0098}" rpy="0 0 0"/>
 			<parent link="Yaw_Link"/>
 			<child link="torso_link"/>
@@ -37,9 +16,4 @@
 			<limit lower="-2.7053" upper="2.7053" effort="30" velocity="5"/>
 		</joint>
-		<joint name="logo_joint" type="fixed">
-			<origin xyz="0.0039635 0 -0.054" rpy="0 0 0"/>
-			<parent link="torso_link"/>
-			<child link="logo_link"/>
-		</joint>
 	</xacro:macro>
 </robot>

File: unitree_g1d_description/xacro/robot.xacro (robot description, xacro)
@@ -6,12 +6,10 @@
 	<xacro:UnitreeG1DChassis/>
 	<xacro:UnitreeG1DBody/>
-	<!-- Shared G1 head (official G1-D mount is 10 mm lower than G1) -->
+	<!-- G1 torso frame: default head / arm mounts (no G1-D mesh offsets) -->
 	<xacro:include filename="$(find unitree_g1_description)/xacro/head.xacro"/>
-	<xacro:UnitreeG1Head xyz_z="-0.054"/>
-	<!-- Shared G1 arms: G1-D torso_link is 9.8 mm higher vs G1 mesh alignment -->
+	<xacro:UnitreeG1Head/>
 	<xacro:include filename="$(find unitree_g1_description)/xacro/arm.xacro"/>
-	<xacro:UnitreeG1Arm name="left" direction="1" mount_xyz_z="-0.0098"/>
-	<xacro:UnitreeG1Arm name="right" direction="-1" mount_xyz_z="-0.0098"/>
-	<!-- Shared G1 end effectors (default Dex3) -->
+	<xacro:UnitreeG1Arm name="left" direction="1"/>
+	<xacro:UnitreeG1Arm name="right" direction="-1"/>
 	<xacro:include filename="$(find unitree_g1_description)/xacro/hand.xacro"/>
 </robot>

File: unitree_g1d_description/xacro/ros2_control/robot.xacro (robot description, xacro)
@@ -43,5 +43,5 @@
 			<state_interface name="velocity"/>
 		</joint>
-		<joint name="torso_Joint">
+		<joint name="torso_yaw_joint">
 			<command_interface name="position"/>
 			<state_interface name="position"/>
