Commit message: Extract shared UnitreeG1Eefs macro for G1, G1-D, and R1-D
Move end-effector selection into eefs.xacro; robot.xacro files call
UnitreeG1Eefs with type. Keep hand.xacro as a thin compatibility shim.

Co-authored-by: Cursor <cursoragent@cursor.com>

File: unitree_g1_description/xacro/hand.xacro (robot description, xacro)
@@ -1,476 +1,8 @@
 <?xml version="1.0" ?>
+<!-- Deprecated: use eefs.xacro / UnitreeG1Eefs. Kept so older includes keep working. -->
 <robot xmlns:xacro="http://www.ros.org/wiki/xacro">
 	<xacro:arg name="type" default="rubber_hand"/>
-	<!-- type:=none — bare wrist, no end effector -->
-	<xacro:if value="${'$(arg type)' == 'none'}">
-	</xacro:if>
-	<xacro:if value="${'$(arg type)' == 'rubber_hand'}">
-		<xacro:macro name="UnitreeG1Hand" params="name direction:=1">
-			<xacro:property name="prefix" value="${name + '_' if name else ''}"/>
-			<!-- Hand Link -->
-			<link name="${prefix}hand_base">
-				<inertial>
-					<origin xyz="0.05361310808 ${direction*-0.00295905240} 0.00215413091"/>
-					<mass value="0.170"/>
-					<inertia ixx="0.00010099485234748" ixy="${direction*0.00003618590790516}"
-												 ixz="-0.00000074301518642" iyy="0.00028135871571621"
-												 iyz="${direction*-0.00000330189743286}" izz="0.00021894770413514"/>
-				</inertial>
-				<visual>
-					<geometry>
-						<mesh filename="file://$(find unitree_g1_description)/meshes/arm/hand.obj" scale="1 ${direction} 1"/>
-					</geometry>
-				</visual>
-				<collision>
-					<origin xyz="0.07 ${direction*-0.02} 0"/>
-					<geometry>
-						<box size="0.12 0.05 0.1"/>
-					</geometry>
-				</collision>
-			</link>
-		</xacro:macro>
-		<xacro:UnitreeG1Hand name="left" direction="1"/>
-		<xacro:UnitreeG1Hand name="right" direction="-1"/>
-		<joint name="left_hand_palm_joint" type="fixed" dont_collapse="true">
-			<origin xyz="0.0415 0.003 0"/>
-			<parent link="left_wrist_yaw_link"/>
-			<child link="left_hand_base"/>
-		</joint>
-		<joint name="right_hand_palm_joint" type="fixed" dont_collapse="true">
-			<origin xyz="0.0415 -0.003 0"/>
-			<parent link="right_wrist_yaw_link"/>
-			<child link="right_hand_base"/>
-		</joint>
-	</xacro:if>
-	<xacro:if value="${'$(arg type)' == 'revo2'}">
-		<xacro:include filename="$(find brainco_description)/xacro/revo2.xacro"/>
-		<xacro:BrainCoHand name="left" direction="1" use_flange="true" fixed_joints="true"/>
-		<xacro:BrainCoHand name="right" direction="-1" use_flange="true" fixed_joints="true"/>
-		<joint name="left_hand_palm_joint" type="fixed" dont_collapse="true">
-			<origin xyz="0.0415 0 0"/>
-			<parent link="left_wrist_yaw_link"/>
-			<child link="left_flange"/>
-		</joint>
-		<joint name="right_hand_palm_joint" type="fixed" dont_collapse="true">
-			<origin xyz="0.0415 0 0"/>
-			<parent link="right_wrist_yaw_link"/>
-			<child link="right_flange"/>
-		</joint>
-	</xacro:if>
-	<xacro:if value="${'$(arg type)' == 'dex3'}">
-		<!-- Dex3 left -->
-		<link name="left_hand_palm_link">
-			<inertial>
-				<origin xyz="0.06214634836 -0.00050869656 -0.00058171093" rpy="0 0 0"/>
-				<mass value="0.37283854"/>
-				<inertia ixx="0.00027535181027" ixy="-0.00001595519465" ixz="-0.00000242161890" iyy="0.00053951827219" iyz="-0.00000042279435" izz="0.00039623390907"/>
-			</inertial>
-			<visual>
-				<origin xyz="0 0 0" rpy="0 0 0"/>
-				<geometry>
-					<mesh filename="file://$(find unitree_g1_description)/meshes/hand/left_hand_palm_link.STL"/>
-				</geometry>
-			</visual>
-			<collision>
-				<origin xyz="0 0 0" rpy="0 0 0"/>
-				<geometry>
-					<mesh filename="file://$(find unitree_g1_description)/meshes/hand/left_hand_palm_link.STL"/>
-				</geometry>
-			</collision>
-		</link>
-		<link name="left_hand_index_0_link">
-			<inertial>
-				<origin xyz="0.03547435774 0.00082788768 0.00038089960" rpy="0 0 0"/>
-				<mass value="0.05885070"/>
-				<inertia ixx="0.00000601573947" ixy="-0.00000050770784" ixz="-0.00000027839003" iyy="0.00001274699945" iyz="0.00000016088850" izz="0.00001234543582"/>
-			</inertial>
-			<visual>
-				<origin xyz="0 0 0" rpy="0 0 0"/>
-				<geometry>
-					<mesh filename="file://$(find unitree_g1_description)/meshes/hand/left_hand_index_0_link.STL"/>
-				</geometry>
-			</visual>
-			<collision>
-				<origin xyz="0 0 0" rpy="0 0 0"/>
-				<geometry>
-					<mesh filename="file://$(find unitree_g1_description)/meshes/hand/left_hand_index_0_link.STL"/>
-				</geometry>
-			</collision>
-		</link>
-		<link name="left_hand_index_1_link">
-			<inertial>
-				<origin xyz="0.02628192939 0.00171735242 -0.00010778879" rpy="0 0 0"/>
-				<mass value="0.02030626"/>
-				<inertia ixx="0.00000153561368" ixy="-0.00000003422130" ixz="-0.00000002549885" iyy="0.00000461267817" iyz="-0.00000000823881" izz="0.00000386625776"/>
-			</inertial>
-			<visual>
-				<origin xyz="0 0 0" rpy="0 0 0"/>
-				<geometry>
-					<mesh filename="file://$(find unitree_g1_description)/meshes/hand/left_hand_index_1_link.STL"/>
-				</geometry>
-			</visual>
-			<collision>
-				<origin xyz="0 0 0" rpy="0 0 0"/>
-				<geometry>
-					<mesh filename="file://$(find unitree_g1_description)/meshes/hand/left_hand_index_1_link.STL"/>
-				</geometry>
-			</collision>
-		</link>
-		<link name="left_hand_middle_0_link">
-			<inertial>
-				<origin xyz="0.03547435774 0.00082788768 0.00038089960" rpy="0 0 0"/>
-				<mass value="0.05885070"/>
-				<inertia ixx="0.00000601573947" ixy="-0.00000050770784" ixz="-0.00000027839003" iyy="0.00001274699945" iyz="0.00000016088850" izz="0.00001234543582"/>
-			</inertial>
-			<visual>
-				<origin xyz="0 0 0" rpy="0 0 0"/>
-				<geometry>
-					<mesh filename="file://$(find unitree_g1_description)/meshes/hand/left_hand_middle_0_link.STL"/>
-				</geometry>
-			</visual>
-			<collision>
-				<origin xyz="0 0 0" rpy="0 0 0"/>
-				<geometry>
-					<mesh filename="file://$(find unitree_g1_description)/meshes/hand/left_hand_middle_0_link.STL"/>
-				</geometry>
-			</collision>
-		</link>
-		<link name="left_hand_middle_1_link">
-			<inertial>
-				<origin xyz="0.02628192939 0.00171735242 -0.00010778879" rpy="0 0 0"/>
-				<mass value="0.02030626"/>
-				<inertia ixx="0.00000153561368" ixy="-0.00000003422130" ixz="-0.00000002549885" iyy="0.00000461267817" iyz="-0.00000000823881" izz="0.00000386625776"/>
-			</inertial>
-			<visual>
-				<origin xyz="0 0 0" rpy="0 0 0"/>
-				<geometry>
-					<mesh filename="file://$(find unitree_g1_description)/meshes/hand/left_hand_middle_1_link.STL"/>
-				</geometry>
-			</visual>
-			<collision>
-				<origin xyz="0 0 0" rpy="0 0 0"/>
-				<geometry>
-					<mesh filename="file://$(find unitree_g1_description)/meshes/hand/left_hand_middle_1_link.STL"/>
-				</geometry>
-			</collision>
-		</link>
-		<link name="left_hand_thumb_0_link">
-			<inertial>
-				<origin xyz="-0.00088424580 -0.00863407079 0.00094429336" rpy="0 0 0"/>
-				<mass value="0.08623657"/>
-				<inertia ixx="0.00001602919238" ixy="0.00000010683177" ixz="0.00000016728875" iyy="0.00001451795012" iyz="-0.00000051094752" izz="0.00001637877663"/>
-			</inertial>
-			<visual>
-				<origin xyz="0 0 0" rpy="0 0 0"/>
-				<geometry>
-					<mesh filename="file://$(find unitree_g1_description)/meshes/hand/left_hand_thumb_0_link.STL"/>
-				</geometry>
-			</visual>
-			<collision>
-				<origin xyz="0 0 0" rpy="0 0 0"/>
-				<geometry>
-					<mesh filename="file://$(find unitree_g1_description)/meshes/hand/left_hand_thumb_0_link.STL"/>
-				</geometry>
-			</collision>
-		</link>
-		<link name="left_hand_thumb_1_link">
-			<inertial>
-				<origin xyz="-0.00082788768 -0.03547435774 -0.00038089960" rpy="0 0 0"/>
-				<mass value="0.05885070"/>
-				<inertia ixx="0.00001274699945" ixy="-0.00000050770784" ixz="0.00000016088850" iyy="0.00000601573947" iyz="-0.00000027839003" izz="0.00001234543582"/>
-			</inertial>
-			<visual>
-				<origin xyz="0 0 0" rpy="0 0 0"/>
-				<geometry>
-					<mesh filename="file://$(find unitree_g1_description)/meshes/hand/left_hand_thumb_1_link.STL"/>
-				</geometry>
-			</visual>
-			<collision>
-				<origin xyz="-0.001 -0.032 0" rpy="0 0 0"/>
-				<geometry>
-					<box size="0.02 0.03 0.02"/>
-				</geometry>
-			</collision>
-		</link>
-		<link name="left_hand_thumb_2_link">
-			<inertial>
-				<origin xyz="-0.00171735242 -0.02628192939 0.00010778879" rpy="0 0 0"/>
-				<mass value="0.02030626"/>
-				<inertia ixx="0.00000461267817" ixy="-0.00000003422130" ixz="-0.00000000823881" iyy="0.00000153561368" iyz="-0.00000002549885" izz="0.00000386625776"/>
-			</inertial>
-			<visual>
-				<origin xyz="0 0 0" rpy="0 0 0"/>
-				<geometry>
-					<mesh filename="file://$(find unitree_g1_description)/meshes/hand/left_hand_thumb_2_link.STL"/>
-				</geometry>
-			</visual>
-			<collision>
-				<origin xyz="0 0 0" rpy="0 0 0"/>
-				<geometry>
-					<mesh filename="file://$(find unitree_g1_description)/meshes/hand/left_hand_thumb_2_link.STL"/>
-				</geometry>
-			</collision>
-		</link>
-		<joint name="left_hand_palm_joint" type="fixed">
-			<origin xyz="0.0415 0.003 0" rpy="0 0 0"/>
-			<parent link="left_wrist_yaw_link"/>
-			<child link="left_hand_palm_link"/>
-		</joint>
-		<joint name="left_hand_index_0_joint" type="revolute">
-			<origin xyz="0.0777 0.0016 0.0285" rpy="0 0 0"/>
-			<parent link="left_hand_palm_link"/>
-			<child link="left_hand_index_0_link"/>
-			<axis xyz="0 0 1"/>
-			<limit lower="-1.57079632" upper="0" effort="1.4" velocity="12"/>
-		</joint>
-		<joint name="left_hand_index_1_joint" type="revolute">
-			<origin xyz="0.0458 0 0" rpy="0 0 0"/>
-			<parent link="left_hand_index_0_link"/>
-			<child link="left_hand_index_1_link"/>
-			<axis xyz="0 0 1"/>
-			<limit lower="-1.74532925" upper="0" effort="1.4" velocity="12"/>
-		</joint>
-		<joint name="left_hand_middle_0_joint" type="revolute">
-			<origin xyz="0.0777 0.0016 -0.0285" rpy="0 0 0"/>
-			<parent link="left_hand_palm_link"/>
-			<child link="left_hand_middle_0_link"/>
-			<axis xyz="0 0 1"/>
-			<limit lower="-1.57079632" upper="0" effort="1.4" velocity="12"/>
-		</joint>
-		<joint name="left_hand_middle_1_joint" type="revolute">
-			<origin xyz="0.0458 0 0" rpy="0 0 0"/>
-			<parent link="left_hand_middle_0_link"/>
-			<child link="left_hand_middle_1_link"/>
-			<axis xyz="0 0 1"/>
-			<limit lower="-1.74532925" upper="0" effort="1.4" velocity="12"/>
-		</joint>
-		<joint name="left_hand_thumb_0_joint" type="revolute">
-			<origin xyz="0.0255 0 0" rpy="0 0 0"/>
-			<parent link="left_hand_palm_link"/>
-			<child link="left_hand_thumb_0_link"/>
-			<axis xyz="0 1 0"/>
-			<limit lower="-1.04719755" upper="1.04719755" effort="2.45" velocity="6.857"/>
-		</joint>
-		<joint name="left_hand_thumb_1_joint" type="revolute">
-			<origin xyz="-0.0025 -0.0193 0" rpy="0 0 0"/>
-			<parent link="left_hand_thumb_0_link"/>
-			<child link="left_hand_thumb_1_link"/>
-			<axis xyz="0 0 1"/>
-			<limit lower="-0.72431163" upper="1.04719755" effort="1.4" velocity="12"/>
-		</joint>
-		<joint name="left_hand_thumb_2_joint" type="revolute">
-			<origin xyz="0 -0.0458 0" rpy="0 0 0"/>
-			<parent link="left_hand_thumb_1_link"/>
-			<child link="left_hand_thumb_2_link"/>
-			<axis xyz="0 0 1"/>
-			<limit lower="0" upper="1.74532925" effort="1.4" velocity="12"/>
-		</joint>
-		<!-- Dex3 right -->
-		<link name="right_hand_palm_link">
-			<inertial>
-				<origin xyz="0.06214634836 0.00050869656 -0.00058171093" rpy="0 0 0"/>
-				<mass value="0.37283854"/>
-				<inertia ixx="0.00027535181027" ixy="0.00001595519465" ixz="-0.00000242161890" iyy="0.00053951827219" iyz="0.00000042279435" izz="0.00039623390907"/>
-			</inertial>
-			<visual>
-				<origin xyz="0 0 0" rpy="0 0 0"/>
-				<geometry>
-					<mesh filename="file://$(find unitree_g1_description)/meshes/hand/right_hand_palm_link.STL"/>
-				</geometry>
-			</visual>
-			<collision>
-				<origin xyz="0 0 0" rpy="0 0 0"/>
-				<geometry>
-					<mesh filename="file://$(find unitree_g1_description)/meshes/hand/right_hand_palm_link.STL"/>
-				</geometry>
-			</collision>
-		</link>
-		<link name="right_hand_index_0_link">
-			<inertial>
-				<origin xyz="0.03547435774 -0.00082788768 0.00038089960" rpy="0 0 0"/>
-				<mass value="0.05885070"/>
-				<inertia ixx="0.00000601573947" ixy="0.00000050770784" ixz="-0.00000027839003" iyy="0.00001274699945" iyz="-0.00000016088850" izz="0.00001234543582"/>
-			</inertial>
-			<visual>
-				<origin xyz="0 0 0" rpy="0 0 0"/>
-				<geometry>
-					<mesh filename="file://$(find unitree_g1_description)/meshes/hand/right_hand_index_0_link.STL"/>
-				</geometry>
-			</visual>
-			<collision>
-				<origin xyz="0 0 0" rpy="0 0 0"/>
-				<geometry>
-					<mesh filename="file://$(find unitree_g1_description)/meshes/hand/right_hand_index_0_link.STL"/>
-				</geometry>
-			</collision>
-		</link>
-		<link name="right_hand_index_1_link">
-			<inertial>
-				<origin xyz="0.02628192939 -0.00171735242 -0.00010778879" rpy="0 0 0"/>
-				<mass value="0.02030626"/>
-				<inertia ixx="0.00000153561368" ixy="0.00000003422130" ixz="-0.00000002549885" iyy="0.00000461267817" iyz="0.00000000823881" izz="0.00000386625776"/>
-			</inertial>
-			<visual>
-				<origin xyz="0 0 0" rpy="0 0 0"/>
-				<geometry>
-					<mesh filename="file://$(find unitree_g1_description)/meshes/hand/right_hand_index_1_link.STL"/>
-				</geometry>
-			</visual>
-			<collision>
-				<origin xyz="0 0 0" rpy="0 0 0"/>
-				<geometry>
-					<mesh filename="file://$(find unitree_g1_description)/meshes/hand/right_hand_index_1_link.STL"/>
-				</geometry>
-			</collision>
-		</link>
-		<link name="right_hand_middle_0_link">
-			<inertial>
-				<origin xyz="0.03547435774 -0.00082788768 0.00038089960" rpy="0 0 0"/>
-				<mass value="0.05885070"/>
-				<inertia ixx="0.00000601573947" ixy="0.00000050770784" ixz="-0.00000027839003" iyy="0.00001274699945" iyz="-0.00000016088850" izz="0.00001234543582"/>
-			</inertial>
-			<visual>
-				<origin xyz="0 0 0" rpy="0 0 0"/>
-				<geometry>
-					<mesh filename="file://$(find unitree_g1_description)/meshes/hand/right_hand_middle_0_link.STL"/>
-				</geometry>
-			</visual>
-			<collision>
-				<origin xyz="0 0 0" rpy="0 0 0"/>
-				<geometry>
-					<mesh filename="file://$(find unitree_g1_description)/meshes/hand/right_hand_middle_0_link.STL"/>
-				</geometry>
-			</collision>
-		</link>
-		<link name="right_hand_middle_1_link">
-			<inertial>
-				<origin xyz="0.02628192939 -0.00171735242 -0.00010778879" rpy="0 0 0"/>
-				<mass value="0.02030626"/>
-				<inertia ixx="0.00000153561368" ixy="0.00000003422130" ixz="-0.00000002549885" iyy="0.00000461267817" iyz="0.00000000823881" izz="0.00000386625776"/>
-			</inertial>
-			<visual>
-				<origin xyz="0 0 0" rpy="0 0 0"/>
-				<geometry>
-					<mesh filename="file://$(find unitree_g1_description)/meshes/hand/right_hand_middle_1_link.STL"/>
-				</geometry>
-			</visual>
-			<collision>
-				<origin xyz="0 0 0" rpy="0 0 0"/>
-				<geometry>
-					<mesh filename="file://$(find unitree_g1_description)/meshes/hand/right_hand_middle_1_link.STL"/>
-				</geometry>
-			</collision>
-		</link>
-		<link name="right_hand_thumb_0_link">
-			<inertial>
-				<origin xyz="-0.00088424580 0.00863407079 0.00094429336" rpy="0 0 0"/>
-				<mass value="0.08623657"/>
-				<inertia ixx="0.00001602919238" ixy="-0.00000010683177" ixz="0.00000016728875" iyy="0.00001451795012" iyz="0.00000051094752" izz="0.00001637877663"/>
-			</inertial>
-			<visual>
-				<origin xyz="0 0 0" rpy="0 0 0"/>
-				<geometry>
-					<mesh filename="file://$(find unitree_g1_description)/meshes/hand/right_hand_thumb_0_link.STL"/>
-				</geometry>
-			</visual>
-			<collision>
-				<origin xyz="0 0 0" rpy="0 0 0"/>
-				<geometry>
-					<mesh filename="file://$(find unitree_g1_description)/meshes/hand/right_hand_thumb_0_link.STL"/>
-				</geometry>
-			</collision>
-		</link>
-		<link name="right_hand_thumb_1_link">
-			<inertial>
-				<origin xyz="-0.00082788768 0.03547435774 -0.00038089960" rpy="0 0 0"/>
-				<mass value="0.05885070"/>
-				<inertia ixx="0.00001274699945" ixy="0.00000050770784" ixz="0.00000016088850" iyy="0.00000601573947" iyz="0.00000027839003" izz="0.00001234543582"/>
-			</inertial>
-			<visual>
-				<origin xyz="0 0 0" rpy="0 0 0"/>
-				<geometry>
-					<mesh filename="file://$(find unitree_g1_description)/meshes/hand/right_hand_thumb_1_link.STL"/>
-				</geometry>
-			</visual>
-			<collision>
-				<origin xyz="-0.001 0.032 0" rpy="0 0 0"/>
-				<geometry>
-					<box size="0.02 0.03 0.02"/>
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
File: unitree_g1_description/xacro/robot.xacro (robot description, xacro)
@@ -1,21 +1,18 @@
+<?xml version="1.0" ?>
 <robot name="g1_29dof" xmlns:xacro="http://www.ros.org/wiki/xacro">
 	<xacro:property name="PI" value="3.1415926535897931"/>
-	<xacro:arg name="end_effector" default="rubber_hand"/>
-	<!-- Include the modular macros -->
+	<xacro:arg name="type" default="rubber_hand"/>
+	<xacro:arg name="eef_fixed_joints" default="false"/>
 	<xacro:include filename="$(find unitree_g1_description)/xacro/arm.xacro"/>
 	<xacro:include filename="$(find unitree_g1_description)/xacro/leg.xacro"/>
 	<xacro:include filename="$(find unitree_g1_description)/xacro/body.xacro"/>
 	<xacro:include filename="$(find unitree_g1_description)/xacro/head.xacro"/>
-	<!-- Legs using modular macro -->
-	<!-- Left leg (direction = 1) -->
+	<xacro:include filename="$(find unitree_g1_description)/xacro/eefs.xacro"/>
 	<xacro:UnitreeG1Leg name="left" direction="1"/>
-	<!-- Right leg (direction = -1 for mirroring) -->
 	<xacro:UnitreeG1Leg name="right" direction="-1"/>
-	<!-- Body using modular macro -->
 	<xacro:UnitreeG1Body/>
 	<xacro:UnitreeG1Head/>
-	<!-- Arms using modular macro -->
 	<xacro:UnitreeG1Arm name="left" direction="1"/>
 	<xacro:UnitreeG1Arm name="right" direction="-1"/>
-	<xacro:include filename="$(find unitree_g1_description)/xacro/hand.xacro"/>
+	<xacro:UnitreeG1Eefs type="$(arg type)" eef_fixed="$(arg eef_fixed_joints)"/>
 </robot>

File: unitree_g1d_description/xacro/robot.xacro (robot description, xacro)
@@ -2,9 +2,9 @@
 <robot name="unitree_g1d" xmlns:xacro="http://www.ros.org/wiki/xacro">
 	<xacro:arg name="type" default="dex3"/>
+	<xacro:arg name="eef_fixed_joints" default="false"/>
 	<xacro:include filename="$(find unitree_g1d_description)/xacro/components/chassis.xacro"/>
 	<xacro:include filename="$(find unitree_g1d_description)/xacro/components/body.xacro"/>
 	<xacro:UnitreeG1DChassis/>
 	<xacro:UnitreeG1DBody/>
-	<!-- G1 torso frame: default head / arm mounts (no G1-D mesh offsets) -->
 	<xacro:include filename="$(find unitree_g1_description)/xacro/head.xacro"/>
 	<xacro:UnitreeG1Head/>
@@ -12,4 +12,5 @@
 	<xacro:UnitreeG1Arm name="left" direction="1"/>
 	<xacro:UnitreeG1Arm name="right" direction="-1"/>
-	<xacro:include filename="$(find unitree_g1_description)/xacro/hand.xacro"/>
+	<xacro:include filename="$(find unitree_g1_description)/xacro/eefs.xacro"/>
+	<xacro:UnitreeG1Eefs type="$(arg type)" eef_fixed="$(arg eef_fixed_joints)"/>
 </robot>

File: unitree_r1d_description/xacro/robot.xacro (robot description, xacro)
@@ -2,9 +2,10 @@
 <robot name="unitree_r1d" xmlns:xacro="http://www.ros.org/wiki/xacro">
 	<xacro:arg name="type" default="none"/>
+	<xacro:arg name="eef_fixed_joints" default="false"/>
 	<xacro:include filename="$(find unitree_r1d_description)/xacro/components/chassis.xacro"/>
 	<xacro:include filename="$(find unitree_r1d_description)/xacro/components/body.xacro"/>
 	<xacro:UnitreeR1DChassis/>
 	<xacro:UnitreeR1DBody/>
-	<!-- Optional end effector from G1 hand macros -->
-	<xacro:include filename="$(find unitree_g1_description)/xacro/hand.xacro"/>
+	<xacro:include filename="$(find unitree_g1_description)/xacro/eefs.xacro"/>
+	<xacro:UnitreeG1Eefs type="$(arg type)" eef_fixed="$(arg eef_fixed_joints)"/>
 </robot>
