Commit message: Use ROS optical frame for G1 D435 (Z forward, X right)
Compose the existing head-camera pitch with (-π/2, 0, -π/2) so
d435_link matches the optical convention used by other humanoids.

Co-authored-by: Cursor <cursoragent@cursor.com>

File: unitree_g1_description/urdf/unitree_g1.urdf (robot description, URDF)
Before this commit: robot g1_29dof, 39 links, 38 joints
Links:
- link head_link: geometry collision mesh filename=file:///home/fiveages/ros2_ws/install/unitree_g1_descriptio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; visual mesh filename=file:///home/fiveages/ros2_ws/install/unitree_g1_descriptio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
- link left_ankle_pitch_link: geometry collision mesh filename=file:///home/fiveages/ros2_ws/install/unitree_g1_descriptio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; visual mesh filename=file:///home/fiveages/ros2_ws/install/unitree_g1_descriptio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
- link left_ankle_roll_link: geometry collision sphere radius=0.005; collision sphere radius=0.005
- link left_elbow_link: geometry collision cylinder length=0.06 radius=0.03; visual mesh filename=file:///home/fiveages/ros2_ws/install/unitree_g1_descriptio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 scale=1 1 1
- link left_hand_base: geometry collision box size=0.12 0.05 0.1; visual mesh filename=file:///home/fiveages/ros2_ws/install/unitree_g1_descriptio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 scale=1 1 1
- link left_hip_pitch_link: geometry collision mesh filename=file:///home/fiveages/ros2_ws/install/unitree_g1_descriptio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 scale=1 1 1; visual mesh filename=file:///home/fiveages/ros2_ws/install/unitree_g1_descriptio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 scale=1 1 1
- link left_hip_roll_link: geometry collision mesh filename=file:///home/fiveages/ros2_ws/install/unitree_g1_descriptio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; visual mesh filename=file:///home/fiveages/ros2_ws/install/unitree_g1_descriptio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
- link left_hip_yaw_link: geometry collision mesh filename=file:///home/fiveages/ros2_ws/install/unitree_g1_descriptio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 scale=1 1 1; visual mesh filename=file:///home/fiveages/ros2_ws/install/unitree_g1_descriptio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 scale=1 1 1
- link left_knee_link: geometry collision mesh filename=file:///home/fiveages/ros2_ws/install/unitree_g1_descriptio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 scale=1 1 1; visual mesh filename=file:///home/fiveages/ros2_ws/install/unitree_g1_descriptio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 scale=1 1 1
- link left_shoulder_pitch_link: geometry collision cylinder length=0.05 radius=0.03; visual mesh filename=file:///home/fiveages/ros2_ws/install/unitree_g1_descriptio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 scale=1 1 1
- link left_shoulder_roll_link: geometry collision cylinder length=0.03 radius=0.03; visual mesh filename=file:///home/fiveages/ros2_ws/install/unitree_g1_descriptio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 scale=1 1 1
- link left_shoulder_yaw_link: geometry collision cylinder length=0.06 radius=0.03; collision cylinder length=0.08 radius=0.03
- link left_wrist_pitch_link: geometry collision cylinder length=0.05 radius=0.03; collision cylinder length=0.06 radius=0.03
- link left_wrist_roll_link: geometry visual mesh filename=file:///home/fiveages/ros2_ws/install/unitree_g1_descriptio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
- link left_wrist_yaw_link: geometry visual mesh filename=file:///home/fiveages/ros2_ws/install/unitree_g1_descriptio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
- link logo_link: geometry visual mesh filename=file:///home/fiveages/ros2_ws/install/unitree_g1_descriptio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
- link pelvis: geometry visual mesh filename=file:///home/fiveages/ros2_ws/install/unitree_g1_descriptio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
- link right_ankle_pitch_link: geometry collision mesh filename=file:///home/fiveages/ros2_ws/install/unitree_g1_descriptio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; visual mesh filename=file:///home/fiveages/ros2_ws/install/unitree_g1_descriptio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
- link right_ankle_roll_link: geometry collision sphere radius=0.005; collision sphere radius=0.005
- link right_elbow_link: geometry collision cylinder length=0.06 radius=0.03; visual mesh filename=file:///home/fiveages/ros2_ws/install/unitree_g1_descriptio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 scale=1 -1 1
- link right_hand_base: geometry collision box size=0.12 0.05 0.1; visual mesh filename=file:///home/fiveages/ros2_ws/install/unitree_g1_descriptio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 scale=1 -1 1
- link right_hip_pitch_link: geometry collision mesh filename=file:///home/fiveages/ros2_ws/install/unitree_g1_descriptio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 scale=1 -1 1; visual mesh filename=file:///home/fiveages/ros2_ws/install/unitree_g1_descriptio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 scale=1 -1 1
- link right_hip_roll_link: geometry collision mesh filename=file:///home/fiveages/ros2_ws/install/unitree_g1_descriptio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; visual mesh filename=file:///home/fiveages/ros2_ws/install/unitree_g1_descriptio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
- link right_hip_yaw_link: geometry collision mesh filename=file:///home/fiveages/ros2_ws/install/unitree_g1_descriptio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 scale=1 -1 1; visual mesh filename=file:///home/fiveages/ros2_ws/install/unitree_g1_descriptio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 scale=1 -1 1
- link right_knee_link: geometry collision mesh filename=file:///home/fiveages/ros2_ws/install/unitree_g1_descriptio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 scale=1 -1 1; visual mesh filename=file:///home/fiveages/ros2_ws/install/unitree_g1_descriptio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 scale=1 -1 1
- link right_shoulder_pitch_link: geometry collision cylinder length=0.05 radius=0.03; visual mesh filename=file:///home/fiveages/ros2_ws/install/unitree_g1_descriptio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 scale=1 -1 1
- link right_shoulder_roll_link: geometry collision cylinder length=0.03 radius=0.03; visual mesh filename=file:///home/fiveages/ros2_ws/install/unitree_g1_descriptio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 scale=1 -1 1
- link right_shoulder_yaw_link: geometry collision cylinder length=0.06 radius=0.03; collision cylinder length=0.08 radius=0.03
- link right_wrist_pitch_link: geometry collision cylinder length=0.05 radius=0.03; collision cylinder length=0.06 radius=0.03
- link right_wrist_roll_link: geometry visual mesh filename=file:///home/fiveages/ros2_ws/install/unitree_g1_descriptio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
- link right_wrist_yaw_link: geometry visual mesh filename=file:///home/fiveages/ros2_ws/install/unitree_g1_descriptio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
- link torso_link: geometry collision box size=0.12 0.15 0.15; collision box size=0.12 0.2 0.15
- link waist_roll_link: geometry visual mesh filename=file:///home/fiveages/ros2_ws/install/unitree_g1_descriptio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
- link waist_yaw_link: geometry visual mesh filename=file:///home/fiveages/ros2_ws/install/unitree_g1_descriptio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
Joints:
- joint d435_joint: origin xyz=0.0576235 0.01753 0.42987 rpy=0 0.8307767239493009 0 -> xyz=0.0576235 0.01753 0.42987 rpy=-2.4015730507441972 0 -1.5707963267948966
