Commit message: Use ROS optical frame for G1 D435 (Z forward, X right)
Compose the existing head-camera pitch with (-π/2, 0, -π/2) so
d435_link matches the optical convention used by other humanoids.

Co-authored-by: Cursor <cursoragent@cursor.com>

File: unitree_g1_description/urdf/unitree_g1_revo2.urdf (robot description, URDF)
Before this commit: robot g1_29dof, 39 links, 38 joints
Links:
- added link left_flange, mass 0.02280635; collision mesh filename=file:///home/fiveages/ros2_ws/install/brainco_description/s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; visual mesh filename=file:///home/fiveages/ros2_ws/install/brainco_description/s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
- added link left_index_distal_Link, mass 0.009; collision mesh filename=file:///home/fiveages/ros2_ws/install/brainco_description/s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; visual mesh filename=file:///home/fiveages/ros2_ws/install/brainco_description/s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
- added link left_index_proximal_Link, mass 0.009; collision mesh filename=file:///home/fiveages/ros2_ws/install/brainco_description/s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; visual mesh filename=file:///home/fiveages/ros2_ws/install/brainco_description/s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
- added link left_index_tip_Link, mass 0.001
- added link left_middle_distal_Link, mass 0.009; collision mesh filename=file:///home/fiveages/ros2_ws/install/brainco_description/s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; visual mesh filename=file:///home/fiveages/ros2_ws/install/brainco_description/s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
- added link left_middle_proximal_Link, mass 0.009; collision mesh filename=file:///home/fiveages/ros2_ws/install/brainco_description/s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; visual mesh filename=file:///home/fiveages/ros2_ws/install/brainco_description/s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
- added link left_middle_tip_Link, mass 0.001
- added link left_pinky_distal_Link, mass 0.009; collision mesh filename=file:///home/fiveages/ros2_ws/install/brainco_description/s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; visual mesh filename=file:///home/fiveages/ros2_ws/install/brainco_description/s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
- added link left_pinky_proximal_Link, mass 0.009; collision mesh filename=file:///home/fiveages/ros2_ws/install/brainco_description/s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; visual mesh filename=file:///home/fiveages/ros2_ws/install/brainco_description/s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
- added link left_pinky_tip_Link, mass 0.001
- added link left_ring_distal_Link, mass 0.009; collision mesh filename=file:///home/fiveages/ros2_ws/install/brainco_description/s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; visual mesh filename=file:///home/fiveages/ros2_ws/install/brainco_description/s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
- added link left_ring_proximal_Link, mass 0.009; collision mesh filename=file:///home/fiveages/ros2_ws/install/brainco_description/s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; visual mesh filename=file:///home/fiveages/ros2_ws/install/brainco_description/s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
- added link left_ring_tip_Link, mass 0.001
- added link left_thumb_distal_Link, mass 0.01; collision mesh filename=file:///home/fiveages/ros2_ws/install/brainco_description/s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; visual mesh filename=file:///home/fiveages/ros2_ws/install/brainco_description/s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
- added link left_thumb_metacarpal_Link, mass 0.01; collision mesh filename=file:///home/fiveages/ros2_ws/install/brainco_description/s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 scale=1 1 1; visual mesh filename=file:///home/fiveages/ros2_ws/install/brainco_description/s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 scale=1 1 1
- added link left_thumb_proximal_Link, mass 0.05; collision mesh filename=file:///home/fiveages/ros2_ws/install/brainco_description/s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; visual mesh filename=file:///home/fiveages/ros2_ws/install/brainco_description/s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
- added link left_thumb_tip_Link, mass 0.001
- added link right_flange, mass 0.02280635; collision mesh filename=file:///home/fiveages/ros2_ws/install/brainco_description/s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; visual mesh filename=file:///home/fiveages/ros2_ws/install/brainco_description/s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
- added link right_index_distal_Link, mass 0.009; collision mesh filename=file:///home/fiveages/ros2_ws/install/brainco_description/s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; visual mesh filename=file:///home/fiveages/ros2_ws/install/brainco_description/s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
- added link right_index_proximal_Link, mass 0.009; collision mesh filename=file:///home/fiveages/ros2_ws/install/brainco_description/s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; visual mesh filename=file:///home/fiveages/ros2_ws/install/brainco_description/s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
- added link right_index_tip_Link, mass 0.001
- added link right_middle_distal_Link, mass 0.009; collision mesh filename=file:///home/fiveages/ros2_ws/install/brainco_description/s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; visual mesh filename=file:///home/fiveages/ros2_ws/install/brainco_description/s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
- added link right_middle_proximal_Link, mass 0.009; collision mesh filename=file:///home/fiveages/ros2_ws/install/brainco_description/s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; visual mesh filename=file:///home/fiveages/ros2_ws/install/brainco_description/s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
- added link right_middle_tip_Link, mass 0.001
- added link right_pinky_distal_Link, mass 0.009; collision mesh filename=file:///home/fiveages/ros2_ws/install/brainco_description/s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; visual mesh filename=file:///home/fiveages/ros2_ws/install/brainco_description/s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
- added link right_pinky_proximal_Link, mass 0.009; collision mesh filename=file:///home/fiveages/ros2_ws/install/brainco_description/s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; visual mesh filename=file:///home/fiveages/ros2_ws/install/brainco_description/s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
- added link right_pinky_tip_Link, mass 0.001
- added link right_ring_distal_Link, mass 0.009; collision mesh filename=file:///home/fiveages/ros2_ws/install/brainco_description/s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; visual mesh filename=file:///home/fiveages/ros2_ws/install/brainco_description/s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
- added link right_ring_proximal_Link, mass 0.009; collision mesh filename=file:///home/fiveages/ros2_ws/install/brainco_description/s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; visual mesh filename=file:///home/fiveages/ros2_ws/install/brainco_description/s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
- added link right_ring_tip_Link, mass 0.001
- added link right_thumb_distal_Link, mass 0.01; collision mesh filename=file:///home/fiveages/ros2_ws/install/brainco_description/s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; visual mesh filename=file:///home/fiveages/ros2_ws/install/brainco_description/s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
- added link right_thumb_metacarpal_Link, mass 0.01; collision mesh filename=file:///home/fiveages/ros2_ws/install/brainco_description/s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 scale=-1 -1 -1; visual mesh filename=file:///home/fiveages/ros2_ws/install/brainco_description/s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 scale=-1 -1 -1
- added link right_thumb_proximal_Link, mass 0.05; collision mesh filename=file:///home/fiveages/ros2_ws/install/brainco_description/s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; visual mesh filename=file:///home/fiveages/ros2_ws/install/brainco_description/s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
- added link right_thumb_tip_Link, mass 0.001
- link head_link: geometry collision mesh filename=file:///home/fiveages/ros2_ws/install/unitree_g1_descriptio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; visual mesh filename=file:///home/fiveages/ros2_ws/install/unitree_g1_descriptio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
- link left_ankle_pitch_link: geometry collision mesh filename=file:///home/fiveages/ros2_ws/install/unitree_g1_descriptio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; visual mesh filename=file:///home/fiveages/ros2_ws/install/unitree_g1_descriptio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
- link left_ankle_roll_link: geometry collision sphere radius=0.005; collision sphere radius=0.005
- link left_elbow_link: geometry collision cylinder length=0.06 radius=0.03; visual mesh filename=file:///home/fiveages/ros2_ws/install/unitree_g1_descriptio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 scale=1 1 1
- link left_hand_base: mass 0.260 -> 0.238; geometry collision mesh filename=file:///home/fiveages/ros2_ws/install/brainco_description/s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 scale=1 1 1; visual mesh filename=file:///home/fiveages/ros2_ws/install/brainco_description/s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 scale=1 1 1
- link left_hip_pitch_link: geometry collision mesh filename=file:///home/fiveages/ros2_ws/install/unitree_g1_descriptio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 scale=1 1 1; visual mesh filename=file:///home/fiveages/ros2_ws/install/unitree_g1_descriptio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 scale=1 1 1
- link left_hip_roll_link: geometry collision mesh filename=file:///home/fiveages/ros2_ws/install/unitree_g1_descriptio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; visual mesh filename=file:///home/fiveages/ros2_ws/install/unitree_g1_descriptio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
- link left_hip_yaw_link: geometry collision mesh filename=file:///home/fiveages/ros2_ws/install/unitree_g1_descriptio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 scale=1 1 1; visual mesh filename=file:///home/fiveages/ros2_ws/install/unitree_g1_descriptio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 scale=1 1 1
- link left_knee_link: geometry collision mesh filename=file:///home/fiveages/ros2_ws/install/unitree_g1_descriptio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 scale=1 1 1; visual mesh filename=file:///home/fiveages/ros2_ws/install/unitree_g1_descriptio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 scale=1 1 1
- link left_shoulder_pitch_link: geometry collision cylinder length=0.05 radius=0.03; visual mesh filename=file:///home/fiveages/ros2_ws/install/unitree_g1_descriptio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 scale=1 1 1
- link left_shoulder_roll_link: geometry collision cylinder length=0.03 radius=0.03; visual mesh filename=file:///home/fiveages/ros2_ws/install/unitree_g1_descriptio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 scale=1 1 1
- link left_shoulder_yaw_link: geometry collision cylinder length=0.06 radius=0.03; collision cylinder length=0.08 radius=0.03
- link left_wrist_pitch_link: geometry collision cylinder length=0.05 radius=0.03; collision cylinder length=0.06 radius=0.03
- link left_wrist_roll_link: geometry visual mesh filename=file:///home/fiveages/ros2_ws/install/unitree_g1_descriptio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
- link left_wrist_yaw_link: geometry visual mesh filename=file:///home/fiveages/ros2_ws/install/unitree_g1_descriptio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
- link logo_link: geometry visual mesh filename=file:///home/fiveages/ros2_ws/install/unitree_g1_descriptio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
- link pelvis: geometry visual mesh filename=file:///home/fiveages/ros2_ws/install/unitree_g1_descriptio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
- link right_ankle_pitch_link: geometry collision mesh filename=file:///home/fiveages/ros2_ws/install/unitree_g1_descriptio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; visual mesh filename=file:///home/fiveages/ros2_ws/install/unitree_g1_descriptio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
- link right_ankle_roll_link: geometry collision sphere radius=0.005; collision sphere radius=0.005
- link right_elbow_link: geometry collision cylinder length=0.06 radius=0.03; visual mesh filename=file:///home/fiveages/ros2_ws/install/unitree_g1_descriptio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 scale=1 -1 1
- link right_hand_base: mass 0.260 -> 0.238; geometry collision mesh filename=file:///home/fiveages/ros2_ws/install/brainco_description/s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 scale=1 -1 1; visual mesh filename=file:///home/fiveages/ros2_ws/install/brainco_description/s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 scale=1 -1 1
- link right_hip_pitch_link: geometry collision mesh filename=file:///home/fiveages/ros2_ws/install/unitree_g1_descriptio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 scale=1 -1 1; visual mesh filename=file:///home/fiveages/ros2_ws/install/unitree_g1_descriptio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 scale=1 -1 1
- link right_hip_roll_link: geometry collision mesh filename=file:///home/fiveages/ros2_ws/install/unitree_g1_descriptio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; visual mesh filename=file:///home/fiveages/ros2_ws/install/unitree_g1_descriptio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
- link right_hip_yaw_link: geometry collision mesh filename=file:///home/fiveages/ros2_ws/install/unitree_g1_descriptio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 scale=1 -1 1; visual mesh filename=file:///home/fiveages/ros2_ws/install/unitree_g1_descriptio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 scale=1 -1 1
- link right_knee_link: geometry collision mesh filename=file:///home/fiveages/ros2_ws/install/unitree_g1_descriptio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 scale=1 -1 1; visual mesh filename=file:///home/fiveages/ros2_ws/install/unitree_g1_descriptio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 scale=1 -1 1
- link right_shoulder_pitch_link: geometry collision cylinder length=0.05 radius=0.03; visual mesh filename=file:///home/fiveages/ros2_ws/install/unitree_g1_descriptio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 scale=1 -1 1
- link right_shoulder_roll_link: geometry collision cylinder length=0.03 radius=0.03; visual mesh filename=file:///home/fiveages/ros2_ws/install/unitree_g1_descriptio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 scale=1 -1 1
- link right_shoulder_yaw_link: geometry collision cylinder length=0.06 radius=0.03; collision cylinder length=0.08 radius=0.03
- link right_wrist_pitch_link: geometry collision cylinder length=0.05 radius=0.03; collision cylinder length=0.06 radius=0.03
- link right_wrist_roll_link: geometry visual mesh filename=file:///home/fiveages/ros2_ws/install/unitree_g1_descriptio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
- link right_wrist_yaw_link: geometry visual mesh filename=file:///home/fiveages/ros2_ws/install/unitree_g1_descriptio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
- link torso_link: geometry collision box size=0.12 0.15 0.15; collision box size=0.12 0.2 0.15
- link waist_roll_link: geometry visual mesh filename=file:///home/fiveages/ros2_ws/install/unitree_g1_descriptio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
- link waist_yaw_link: geometry visual mesh filename=file:///home/fiveages/ros2_ws/install/unitree_g1_descriptio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
Joints:
- added joint left_flange_joint: type fixed, parent left_flange, child left_hand_base, origin xyz=0.0176 0 0 rpy=-1.570796326 0 -1.570796326
- added joint left_index_distal_joint: type fixed, parent left_index_proximal_Link, child left_index_distal_Link, origin xyz=0 0 0.032
- added joint left_index_joint: type fixed, parent left_hand_base, child left_index_proximal_Link, origin xyz=-0.0021349 -0.029578 0.080876 rpy=0.11819 0.14743 0.17422
- added joint left_index_tip_joint: type fixed, parent left_index_distal_Link, child left_index_tip_Link, origin xyz=0.011097 0 0.035739 rpy=0 0.48723 0
- added joint left_middle_distal_joint: type fixed, parent left_middle_proximal_Link, child left_middle_distal_Link, origin xyz=0 0 0.037 rpy=0 0.12654 0
- added joint left_middle_joint: type fixed, parent left_hand_base, child left_middle_proximal_Link, origin xyz=-0.0045935 -0.010061 0.084993 rpy=0.039468 0.1483 0.057975
- added joint left_middle_tip_joint: type fixed, parent left_middle_distal_Link, child left_middle_tip_Link, origin xyz=0.0073534 0 0.041703 rpy=0 0.34907 0
- added joint left_pinky_distal_joint: type fixed, parent left_pinky_proximal_Link, child left_pinky_distal_Link, origin xyz=0 0 0.029
- added joint left_pinky_joint: type fixed, parent left_hand_base, child left_pinky_proximal_Link, origin xyz=-0.0023733 0.029356 0.078694 rpy=-0.11815 0.14491 -0.17392
- added joint left_pinky_tip_joint: type fixed, parent left_pinky_distal_Link, child left_pinky_tip_Link, origin xyz=0.010221 0 0.032918 rpy=0 0.4756 0
- added joint left_ring_distal_joint: type fixed, parent left_ring_proximal_Link, child left_ring_distal_Link, origin xyz=0 0 0.035 rpy=0 0.12654 0
- added joint left_ring_joint: type fixed, parent left_hand_base, child left_ring_proximal_Link, origin xyz=-0.00468767815858587 0.0100262714211602 0.0839819548795939 rpy=-0.0394618478609065 0.147209177132223 -0.0579317909005277
- added joint left_ring_tip_joint: type fixed, parent left_ring_distal_Link, child left_ring_tip_Link, origin xyz=0.0071824 0 0.040734 rpy=0 0.34907 0
- added joint left_thumb_distal_joint: type fixed, parent left_thumb_proximal_Link, child left_thumb_distal_Link, origin xyz=0 0.052 0
- added joint left_thumb_joint1: type fixed, parent left_thumb_metacarpal_Link, child left_thumb_proximal_Link, origin xyz=0 -0.014227 0 rpy=0.17488 -0.23736 2.9737
- added joint left_thumb_joint2: type fixed, parent left_hand_base, child left_thumb_metacarpal_Link, origin xyz=0.0045 -0.019 0.027825 rpy=0.0 0 0.16787
- added joint left_thumb_tip_joint: type fixed, parent left_thumb_distal_Link, child left_thumb_tip_Link, origin xyz=0 0.026528781163583 -0.00177344281307927 rpy=0.0667504507189052 0 3.14159265358979
- added joint right_flange_joint: type fixed, parent right_flange, child right_hand_base, origin xyz=0.0176 0 0 rpy=1.570796326 0 1.570796326
- added joint right_index_distal_joint: type fixed, parent right_index_proximal_Link, child right_index_distal_Link, origin xyz=0 0 0.032
- added joint right_index_joint: type fixed, parent right_hand_base, child right_index_proximal_Link, origin xyz=-0.0021349 0.029578 0.080876 rpy=-0.11819 0.14743 -0.17422
- added joint right_index_tip_joint: type fixed, parent right_index_distal_Link, child right_index_tip_Link, origin xyz=0.011097 0 0.035739 rpy=0 0.48723 0
- added joint right_middle_distal_joint: type fixed, parent right_middle_proximal_Link, child right_middle_distal_Link, origin xyz=0 0 0.037 rpy=0 0.12654 0
- added joint right_middle_joint: type fixed, parent right_hand_base, child right_middle_proximal_Link, origin xyz=-0.0045935 0.010061 0.084993 rpy=-0.039468 0.1483 -0.057975
- added joint right_middle_tip_joint: type fixed, parent right_middle_distal_Link, child right_middle_tip_Link, origin xyz=0.0073534 0 0.041703 rpy=0 0.34907 0
- added joint right_pinky_distal_joint: type fixed, parent right_pinky_proximal_Link, child right_pinky_distal_Link, origin xyz=0 0 0.029
- added joint right_pinky_joint: type fixed, parent right_hand_base, child right_pinky_proximal_Link, origin xyz=-0.0023733 -0.029356 0.078694 rpy=0.11815 0.14491 0.17392
- added joint right_pinky_tip_joint: type fixed, parent right_pinky_distal_Link, child right_pinky_tip_Link, origin xyz=0.010221 0 0.032918 rpy=0 0.4756 0
- added joint right_ring_distal_joint: type fixed, parent right_ring_proximal_Link, child right_ring_distal_Link, origin xyz=0 0 0.035 rpy=0 0.12654 0
- added joint right_ring_joint: type fixed, parent right_hand_base, child right_ring_proximal_Link, origin xyz=-0.00468767815858587 -0.0100262714211602 0.0839819548795939 rpy=0.0394618478609065 0.147209177132223 0.0579317909005277
- added joint right_ring_tip_joint: type fixed, parent right_ring_distal_Link, child right_ring_tip_Link, origin xyz=0.0071824 0 0.040734 rpy=0 0.34907 0
- added joint right_thumb_distal_joint: type fixed, parent right_thumb_proximal_Link, child right_thumb_distal_Link, origin xyz=0 0.052 0
- added joint right_thumb_joint1: type fixed, parent right_thumb_metacarpal_Link, child right_thumb_proximal_Link, origin xyz=0 0.014227 0 rpy=-2.9667 -0.23736 2.9737
- added joint right_thumb_joint2: type fixed, parent right_hand_base, child right_thumb_metacarpal_Link, origin xyz=0.005619 0.019867 0.027825 rpy=3.1416 0 2.9637
- added joint right_thumb_tip_joint: type fixed, parent right_thumb_distal_Link, child right_thumb_tip_Link, origin xyz=0 0.026528781163583 -0.00177344281307927 rpy=-0.06675 0 0
- joint d435_joint: origin xyz=0.0576235 0.01753 0.42987 rpy=0 0.8307767239493009 0 -> xyz=0.0576235 0.01753 0.42987 rpy=-2.4015730507441972 0 -1.5707963267948966
- joint left_hand_palm_joint: child left_hand_base -> left_flange; origin xyz=0.0415 0.003 0 -> xyz=0.0415 0 0
- joint right_hand_palm_joint: child right_hand_base -> right_flange; origin xyz=0.0415 -0.003 0 -> xyz=0.0415 0 0

File: unitree_g1_description/xacro/torso.xacro (robot description, xacro)
@@ -1,4 +1,5 @@
 <?xml version="1.0" ?>
 <robot xmlns:xacro="http://www.ros.org/wiki/xacro">
+	<xacro:property name="PI" value="3.1415926535897931"/>
 	<!--
 	G1 torso + logo + torso-mounted sensors.
@@ -53,7 +54,10 @@
 			<child link="imu_in_torso"/>
 		</joint>
+		<!-- D435: ROS optical (+Z forward, +X right, +Y down). Mount pitch 0.8308
+		     was previously X-forward/Z-up; compose with (-PI/2, 0, -PI/2). -->
 		<link name="d435_link"/>
 		<joint name="d435_joint" type="fixed">
-			<origin xyz="0.0576235 0.01753 0.42987" rpy="0 0.8307767239493009 0"/>
+			<origin xyz="0.0576235 0.01753 0.42987"
+							rpy="${-PI/2 - 0.8307767239493009} 0 ${-PI/2}"/>
 			<parent link="torso_link"/>
 			<child link="d435_link"/>
