Commit message: update unitree config

File: unitree_dex_description/xacro/dex3.xacro (robot description, xacro)
@@ -3,5 +3,7 @@
   Unitree Dex3 hand (one side). name="left"/"right"; direction 1=left, -1=right.
   One mesh set (left CAD). Right side places each mesh with rpy=π about X.
-  Kinematics and inertials use Y-mirror via direction. Palm mount stays on the robot.
+  Link origins / inertials use Y-mirror via direction for placement only.
+  Joint limits and joint-angle semantics are identical on both sides (not mirrored):
+  the same home / command vector is valid for left and right.
   OCS2 planning: robot_common_launch injects eef_fixed_joints:=true → finger joints
   become fixed (same as Revo1/Revo2); do not list them in .info removeJoints.
@@ -184,6 +186,5 @@
             <xacro:unless value="${joints_are_fixed}">
                 <axis xyz="0 0 1"/>
-                <limit lower="${-1.57079632 if dir > 0 else 0}" upper="${0 if dir > 0 else 1.57079632}"
-                       effort="1.4" velocity="12"/>
+                <limit lower="-1.57079632" upper="0" effort="1.4" velocity="12"/>
             </xacro:unless>
         </joint>
@@ -194,6 +195,5 @@
             <xacro:unless value="${joints_are_fixed}">
                 <axis xyz="0 0 1"/>
-                <limit lower="${-1.74532925 if dir > 0 else 0}" upper="${0 if dir > 0 else 1.74532925}"
-                       effort="1.4" velocity="12"/>
+                <limit lower="-1.74532925" upper="0" effort="1.4" velocity="12"/>
             </xacro:unless>
         </joint>
@@ -204,6 +204,5 @@
             <xacro:unless value="${joints_are_fixed}">
                 <axis xyz="0 0 1"/>
-                <limit lower="${-1.57079632 if dir > 0 else 0}" upper="${0 if dir > 0 else 1.57079632}"
-                       effort="1.4" velocity="12"/>
+                <limit lower="-1.57079632" upper="0" effort="1.4" velocity="12"/>
             </xacro:unless>
         </joint>
@@ -214,6 +213,5 @@
             <xacro:unless value="${joints_are_fixed}">
                 <axis xyz="0 0 1"/>
-                <limit lower="${-1.74532925 if dir > 0 else 0}" upper="${0 if dir > 0 else 1.74532925}"
-                       effort="1.4" velocity="12"/>
+                <limit lower="-1.74532925" upper="0" effort="1.4" velocity="12"/>
             </xacro:unless>
         </joint>
@@ -233,8 +231,5 @@
             <xacro:unless value="${joints_are_fixed}">
                 <axis xyz="0 0 1"/>
-                <!-- left [-0.724, 1.047]; right is negate+swap -->
-                <limit lower="${-0.72431163 if dir > 0 else -1.04719755}"
-                       upper="${1.04719755 if dir > 0 else 0.72431163}"
-                       effort="1.4" velocity="12"/>
+                <limit lower="-0.72431163" upper="1.04719755" effort="1.4" velocity="12"/>
             </xacro:unless>
         </joint>
@@ -245,6 +240,5 @@
             <xacro:unless value="${joints_are_fixed}">
                 <axis xyz="0 0 1"/>
-                <limit lower="${0 if dir > 0 else -1.74532925}" upper="${1.74532925 if dir > 0 else 0}"
-                       effort="1.4" velocity="12"/>
+                <limit lower="0" upper="1.74532925" effort="1.4" velocity="12"/>
             </xacro:unless>
         </joint>

File: unitree_g1_description/xacro/eefs.xacro (robot description, xacro)
@@ -4,4 +4,5 @@
 	Shared end effectors for Unitree G1 / G1-D / H2D.
 	type: none | rubber_hand | revo2 | dex3 | dex1
+	left_type / right_type override one side (W2-style). Empty side falls back to type.
 	Parent frames: left/right_tcp (flange on UnitreeG1Arm).
 	eef_fixed: OCS2 planning injects eef_fixed_joints:=true (robot_common_launch);
@@ -10,89 +11,72 @@
 	<xacro:include filename="$(find unitree_dex_description)/xacro/dex1.xacro"/>
 	<xacro:include filename="$(find unitree_dex_description)/xacro/dex3.xacro"/>
-	<xacro:macro name="UnitreeG1Eefs" params="type:=rubber_hand eef_fixed:=false camera:=false">
-		<xacro:if value="${type == 'none'}">
-			<!-- bare flange: left/right_tcp from the arm -->
+	<xacro:macro name="UnitreeG1Hand" params="name direction:=1">
+		<xacro:property name="prefix" value="${name + '_' if name else ''}"/>
+		<link name="${prefix}hand_base">
+			<inertial>
+				<origin xyz="0.05361310808 ${direction*-0.00295905240} 0.00215413091"/>
+				<mass value="0.170"/>
+				<inertia ixx="0.00010099485234748" ixy="${direction*0.00003618590790516}"
+											 ixz="-0.00000074301518642" iyy="0.00028135871571621"
+											 iyz="${direction*-0.00000330189743286}" izz="0.00021894770413514"/>
+			</inertial>
+			<visual>
+				<geometry>
+					<mesh filename="file://$(find unitree_g1_description)/meshes/arm/hand.glb" scale="1 ${direction} 1"/>
+				</geometry>
+			</visual>
+			<collision>
+				<origin xyz="0.07 ${direction*-0.02} 0"/>
+				<geometry>
+					<box size="0.12 0.05 0.1"/>
+				</geometry>
+			</collision>
+		</link>
+	</xacro:macro>
+	<xacro:macro name="UnitreeG1EefSide" params="side direction ee eef_fixed camera">
+		<xacro:if value="${ee == 'none' or ee == ''}">
+			<!-- bare flange: ${side}_tcp from the arm -->
 		</xacro:if>
-	<xacro:if value="${type == 'rubber_hand'}">
-			<xacro:macro name="UnitreeG1Hand" params="name direction:=1">
-				<xacro:property name="prefix" value="${name + '_' if name else ''}"/>
-				<!-- Hand Link -->
-				<link name="${prefix}hand_base">
-					<inertial>
-						<origin xyz="0.05361310808 ${direction*-0.00295905240} 0.00215413091"/>
-						<mass value="0.170"/>
-						<inertia ixx="0.00010099485234748" ixy="${direction*0.00003618590790516}"
-													 ixz="-0.00000074301518642" iyy="0.00028135871571621"
-													 iyz="${direction*-0.00000330189743286}" izz="0.00021894770413514"/>
-					</inertial>
-					<visual>
-						<geometry>
-							<mesh filename="file://$(find unitree_g1_description)/meshes/arm/hand.glb" scale="1 ${direction} 1"/>
-						</geometry>
-					</visual>
-					<collision>
-						<origin xyz="0.07 ${direction*-0.02} 0"/>
-						<geometry>
-							<box size="0.12 0.05 0.1"/>
-						</geometry>
-					</collision>
-				</link>
-			</xacro:macro>
-			<xacro:UnitreeG1Hand name="left" direction="1"/>
-			<xacro:UnitreeG1Hand name="right" direction="-1"/>
-			<joint name="left_hand_palm_joint" type="fixed" dont_collapse="true">
-				<origin xyz="0 0.003 0"/>
-				<parent link="left_tcp"/>
-				<child link="left_hand_base"/>
-			</joint>
-			<joint name="right_hand_palm_joint" type="fixed" dont_collapse="true">
-				<origin xyz="0 -0.003 0"/>
-				<parent link="right_tcp"/>
-				<child link="right_hand_base"/>
+		<xacro:if value="${ee == 'rubber_hand'}">
+			<xacro:UnitreeG1Hand name="${side}" direction="${direction}"/>
+			<joint name="${side}_hand_palm_joint" type="fixed" dont_collapse="true">
+				<origin xyz="0 ${direction * 0.003} 0"/>
+				<parent link="${side}_tcp"/>
+				<child link="${side}_hand_base"/>
 			</joint>
 		</xacro:if>
-		<xacro:if value="${type == 'revo2'}">
-			<xacro:include filename="$(find brainco_description)/xacro/revo2.xacro"/>
-			<xacro:BrainCoHand name="left" direction="1" use_flange="true" fixed_joints="${eef_fixed}"/>
-			<xacro:BrainCoHand name="right" direction="-1" use_flange="true" fixed_joints="${eef_fixed}"/>
-			<joint name="left_hand_palm_joint" type="fixed" dont_collapse="true">
+		<xacro:if value="${ee == 'revo2'}">
+			<xacro:BrainCoHand name="${side}_hand" direction="${direction}" use_flange="true" fixed_joints="${eef_fixed}"/>
+			<joint name="${side}_hand_palm_joint" type="fixed" dont_collapse="true">
 				<origin xyz="0 0 0"/>
-				<parent link="left_tcp"/>
-				<child link="left_flange"/>
-			</joint>
-			<joint name="right_hand_palm_joint" type="fixed" dont_collapse="true">
-				<origin xyz="0 0 0"/>
-				<parent link="right_tcp"/>
-				<child link="right_flange"/>
+				<parent link="${side}_tcp"/>
+				<child link="${side}_hand_flange"/>
 			</joint>
 		</xacro:if>
-		<xacro:if value="${type == 'dex3'}">
-			<xacro:UnitreeDex3 name="left" direction="1" fixed_joints="${eef_fixed}"/>
-			<xacro:UnitreeDex3 name="right" direction="-1" fixed_joints="${eef_fixed}"/>
-			<joint name="left_hand_palm_joint" type="fixed">
-				<origin xyz="0 0.003 0" rpy="0 0 0"/>
-				<parent link="left_tcp"/>
-				<child link="left_hand_palm_link"/>
-			</joint>
-			<joint name="right_hand_palm_joint" type="fixed">
-				<origin xyz="0 -0.003 0" rpy="0 0 0"/>
-				<parent link="right_tcp"/>
-				<child link="right_hand_palm_link"/>
+		<xacro:if value="${ee == 'dex3'}">
+			<xacro:UnitreeDex3 name="${side}" direction="${direction}" fixed_joints="${eef_fixed}"/>
+			<joint name="${side}_hand_palm_joint" type="fixed">
+				<origin xyz="0 ${direction * 0.003} 0" rpy="0 0 0"/>
+				<parent link="${side}_tcp"/>
+				<child link="${side}_hand_palm_link"/>
 			</joint>
 		</xacro:if>
-		<xacro:if value="${type == 'dex1'}">
-			<xacro:UnitreeDex1 name="left" eef_fixed="${eef_fixed}" camera="${camera}"/>
-			<xacro:UnitreeDex1 name="right" eef_fixed="${eef_fixed}" camera="${camera}"/>
-			<joint name="left_base_joint" type="fixed">
+		<xacro:if value="${ee == 'dex1'}">
+			<xacro:UnitreeDex1 name="${side}" eef_fixed="${eef_fixed}" camera="${camera}"/>
+			<joint name="${side}_base_joint" type="fixed">
 				<origin xyz="0 0 0"/>
-				<parent link="left_tcp"/>
-				<child link="left_dex1_base_link"/>
-			</joint>
-			<joint name="right_base_joint" type="fixed">
-				<origin xyz="0 0 0"/>
-				<parent link="right_tcp"/>
-				<child link="right_dex1_base_link"/>
+				<parent link="${side}_tcp"/>
+				<child link="${side}_dex1_base_link"/>
 			</joint>
 		</xacro:if>
 	</xacro:macro>
+	<xacro:macro name="UnitreeG1Eefs" params="type:=rubber_hand left_type:='' right_type:='' eef_fixed:=false camera:=false">
+		<xacro:property name="ee_left" value="${left_type if left_type != '' else type}"/>
+		<xacro:property name="ee_right" value="${right_type if right_type != '' else type}"/>
+		<xacro:if value="${ee_left == 'revo2' or ee_right == 'revo2'}">
+			<xacro:include filename="$(find brainco_description)/xacro/revo2.xacro"/>
+		</xacro:if>
+		<xacro:UnitreeG1EefSide side="left" direction="1" ee="${ee_left}" eef_fixed="${eef_fixed}" camera="${camera}"/>
+		<xacro:UnitreeG1EefSide side="right" direction="-1" ee="${ee_right}" eef_fixed="${eef_fixed}" camera="${camera}"/>
+	</xacro:macro>
 </robot>

File: unitree_g1d_description/xacro/robot.xacro (robot description, xacro)
@@ -1,7 +1,10 @@
 <?xml version="1.0"?>
 <robot name="unitree_g1d" xmlns:xacro="http://www.ros.org/wiki/xacro">
-	<!-- type: none | rubber_hand | revo2 | dex3 | dex1
+	<!-- type: none | rubber_hand | revo2 | dex3 | dex1 (both sides).
+	     left_type / right_type override one side, same as FiveAges W2.
 	     OCS2 planning: robot_common_launch injects eef_fixed_joints:=true. -->
 	<xacro:arg name="type" default="dex3"/>
+	<xacro:arg name="left_type" default=""/>
+	<xacro:arg name="right_type" default=""/>
 	<xacro:arg name="eef_fixed_joints" default="false"/>
 	<!-- Dex1 optional wrist camera mount + optical frame. -->
@@ -23,4 +26,4 @@
 	<xacro:UnitreeG1Arm name="right" direction="-1"/>
 	<xacro:include filename="$(find unitree_g1_description)/xacro/eefs.xacro"/>
-	<xacro:UnitreeG1Eefs type="$(arg type)" eef_fixed="$(arg eef_fixed_joints)" camera="$(arg camera)"/>
+	<xacro:UnitreeG1Eefs type="$(arg type)" left_type="$(arg left_type)" right_type="$(arg right_type)" eef_fixed="$(arg eef_fixed_joints)" camera="$(arg camera)"/>
 </robot>

File: unitree_g1d_description/xacro/ros2_control/robot.xacro (robot description, xacro)
@@ -7,4 +7,22 @@
 	<xacro:include filename="$(find unitree_dex_description)/xacro/ros2_control/dex1.xacro"/>
 	<xacro:include filename="$(find unitree_dex_description)/xacro/ros2_control/dex3.xacro"/>
+	<xacro:include filename="$(find brainco_description)/xacro/ros2_control/revo2.xacro"/>
+	<!-- Same fallback as UnitreeG1Eefs: empty side arg uses type. -->
+	<xacro:property name="g1d_type" value="$(arg type)"/>
+	<xacro:property name="g1d_left_arg" value="$(arg left_type)"/>
+	<xacro:property name="g1d_right_arg" value="$(arg right_type)"/>
+	<xacro:property name="g1d_left_ee" value="${g1d_left_arg if g1d_left_arg != '' else g1d_type}"/>
+	<xacro:property name="g1d_right_ee" value="${g1d_right_arg if g1d_right_arg != '' else g1d_type}"/>
+	<xacro:macro name="UnitreeG1DEefInterfaces" params="side ee">
+		<xacro:if value="${ee == 'dex1'}">
+			<xacro:UnitreeDex1Interfaces name="${side}" eef_fixed="$(arg eef_fixed_joints)"/>
+		</xacro:if>
+		<xacro:if value="${ee == 'dex3'}">
+			<xacro:UnitreeDex3Interfaces name="${side}" eef_fixed="$(arg eef_fixed_joints)"/>
+		</xacro:if>
+		<xacro:if value="${ee == 'revo2'}">
+			<xacro:revo2_interfaces name="${side}_hand"/>
+		</xacro:if>
+	</xacro:macro>
 	<ros2_control name="unitree_g1d_system" type="system">
 		<hardware>
@@ -67,15 +85,9 @@
 			<state_interface name="effort"/>
 		</joint>
-		<!-- Arms (unitree_g1_description). Dex1 / Dex3 (unitree_dex_description). -->
+		<!-- Arms (unitree_g1_description). Per-side Dex1 / Dex3 / Revo2. -->
 		<xacro:UnitreeG1ArmInterfaces name="left"/>
 		<xacro:UnitreeG1ArmInterfaces name="right"/>
-		<xacro:if value="${'$(arg type)' == 'dex1'}">
-			<xacro:UnitreeDex1Interfaces name="left" eef_fixed="$(arg eef_fixed_joints)"/>
-			<xacro:UnitreeDex1Interfaces name="right" eef_fixed="$(arg eef_fixed_joints)"/>
-		</xacro:if>
-		<xacro:if value="${'$(arg type)' == 'dex3'}">
-			<xacro:UnitreeDex3Interfaces name="left" eef_fixed="$(arg eef_fixed_joints)"/>
-			<xacro:UnitreeDex3Interfaces name="right" eef_fixed="$(arg eef_fixed_joints)"/>
-		</xacro:if>
+		<xacro:UnitreeG1DEefInterfaces side="left" ee="${g1d_left_ee}"/>
+		<xacro:UnitreeG1DEefInterfaces side="right" ee="${g1d_right_ee}"/>
 	</ros2_control>
 	<xacro:if value="$(arg gazebo)">
